File: dist/manufacturing/kicad-project/pd1180-epr-r0.3.kicad_pcb (KiCad board)
At the start: 4 copper layers, 85.9 x 85.9 mm, 255 parts, among them J1 J1, J2 J2, J3 J3, J4 J4, J5 J5, J6 J6, J7 J7, J8 J8, J9 J9, Q1 BSS123LT1G, Q10 CSD19534Q5A, Q11 CSD19534Q5A, Q12 CSD19534Q5A, Q13 CSD19534Q5A, Q14 MMBT5551LT1G, Q15 MMBT5551LT1G, Q16 CSD19534Q5A, Q17 MMBT5551LT1G, Q18 MMBT5551LT1G, Q19 MMBT5551LT1G, Q2 MMBT5551LT1G, Q20 MMBT5551LT1G, Q21 MMBT5551LT1G, Q22 MMBT5551LT1G, Q23 MMBT5551LT1G, Q24 MMBT5551LT1G, Q25 MMBT5551LT1G, Q3 MMBT5551LT1G, Q4 CSD19534Q5A, Q5 BSS123LT1G, Q6 CSD19534Q5A, Q7 CSD19534Q5A, Q8 CSD19534Q5A, Q9 CSD19534Q5A, SW1 SW1, U1 TPD4S480RUKR, U10 SN74LVC1G08DBVR, U11 SN74LVC1G08DBVR, U12 TL431AIDBZR, U13 TLV3201AIDBVR, U14 TLV3201AIDBVR, U15 UCC27511DBVR, U16 STM32G0B1CBT6, U17 W25Q32JVSSIQ, U18 AS5047P-ATSM, U19 TCAN332DR, U2 TPS26750SRSMR, U20 MAX3485EESA+T, U21 MAX3232ESE+T, U22 LMR36510ADDAR, U23 LM66100DCKR, U24 LM66100DCKR, U3 M24512-RMN6TP, U4 SN74LVC1G08DBVR, U5 LMR36510ADDAR, U6 TPS26631RGER, U7 TMC5160A-TA-T, U8 74LVC1G157GW,125, U9 74LVC1G157GW,125, Y1 Y1

Commit message: Add full product name to PCB silkscreen
Other:
- board text added: "PD1180-EPR — NEMA 34 Smart Motor-Mounted"
- board text added: "Stepper Controller with USB-C PD 3.1 EPR · r0.3"
- board text removed: "48V EPR CONTROLLER"
- board text removed: "PD1180-EPR r0.3"
Changed lines of the file:
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@@
 		)
 	)
-	(gr_text "48V EPR CONTROLLER"
+	(gr_text "Stepper Controller with USB-C PD 3.1 EPR · r0.3"
 		(at 100 59.5 0)
 		(layer "F.SilkS")
@@
 		)
 	)
-	(gr_text "PD1180-EPR r0.3"
+	(gr_text "PD1180-EPR — NEMA 34 Smart Motor-Mounted"
 		(at 100 58.2 0)
 		(layer "F.SilkS")
 		(effects
 			(font
-				(size 1 1)
-				(thickness 0.15)
-			)
+				(size 0.8 0.8)
+				(thickness 0.15)
+			)

Commit message: Add reusable PCB review and delivery gates
Other:
- board text added: "Made with tscircuit"
- board text added: "ts"
Changed lines of the file:
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@@
+		)
+	)
+	(gr_text "ts"
+		(at 100 96 0)
+		(layer "B.SilkS")
+		(effects
+			(font
+				(size 2.4 2.4)
+				(thickness 0.35)
+			)
+			(justify mirror)
+		)
+	)
+	(gr_text "Made with tscircuit"
+		(at 100 98.5 0)
+		(layer "B.SilkS")
+		(effects
+			(font
+				(size 0.9 0.9)
+				(thickness 0.15)
+			)
+			(justify mirror)
 		)
 	)

Commit message: Complete orderable PD1180-EPR board release
Parts:
- removed J4: J4, tscircuit:B6B-PH-K-S_LF_SN
- removed J5: J5, tscircuit:B5B-PH-K-S_LF_SN
- removed J8: J8, tscircuit:B4B-PH-K-S_LF_SN
- removed MH1, MH2, MH3, MH4: , tscircuit:hole_circle_holeDiameter4.2mm
- removed RS1, RS2: HoLLR2512-3W-33mR-1%, tscircuit:HoLLR2512-3W-33mR-1
- added ?: , hole_circle_holeDiameter4.2mm, F.Cu at (75.5, 138.4)
- added ?: , hole_circle_holeDiameter4.2mm, F.Cu at (138.4, 124.5)
- added ?: , hole_circle_holeDiameter4.2mm, F.Cu at (61.6, 75.5)
- added ?: , hole_circle_holeDiameter4.2mm, F.Cu at (124.5, 61.6)
- added C72: 100nF, capacitor_cap0603, F.Cu at (77.0, 86.0)
- added J10: J10, USB4105-GF-A, F.Cu at (63.6, 98.0)
- added R105: 5.1kΩ, resistor_res0603, F.Cu at (69.0, 80.5)
- added R106: 5.1kΩ, resistor_res0603, F.Cu at (68.5, 86.0)
- added R107: 100kΩ, resistor_res0603, F.Cu at (78.0, 84.0)
- added R108: 100kΩ, resistor_res0603, F.Cu at (81.0, 84.0)
- added R109: 33mΩ, HoLLR2512-3W-33mR-1, F.Cu at (120.0, 124.0)
- added R110: 33mΩ, HoLLR2512-3W-33mR-1, F.Cu at (131.0, 124.0)
- added TP_ENC_3V3: TP_ENC_3V3, test_point, B.Cu at (88.0, 134.0)
- added TP_ENC_A: TP_ENC_A, test_point, B.Cu at (91.0, 134.0)
- added TP_ENC_B: TP_ENC_B, test_point, B.Cu at (94.0, 134.0)
- added TP_ENC_GND: TP_ENC_GND, test_point, B.Cu at (100.0, 134.0)
- added TP_ENC_I: TP_ENC_I, test_point, B.Cu at (97.0, 134.0)
- added TP_NRST: TP_NRST, test_point, B.Cu at (83.0, 130.0)
- added TP_STATUS: TP_STATUS, test_point, B.Cu at (86.0, 130.0)
- added TP_SWCLK: TP_SWCLK, test_point, B.Cu at (80.0, 130.0)
- added TP_SWDIO: TP_SWDIO, test_point, B.Cu at (83.0, 133.0)
- added TP_SWD_3V3: TP_SWD_3V3, test_point, B.Cu at (80.0, 133.0)
- added TP_SWD_GND: TP_SWD_GND, test_point, B.Cu at (86.0, 133.0)
- C1, C12, C13, C14, C26, C52, C53, C71: footprint tscircuit:capacitor_cap0603 -> capacitor_cap0603; moved to B.Cu
- C10, C18, C19, C2, C20, C24, C28, C29, C3, C31, C36, C37, C38, C39, C4, C40, C41, C42, C43, C44, C45, C46, C48, C49, C50, C51, C54, C55, C56, C57, C58, C59, C6, C60, C61, C63, C64, C65, C69, C7, C70, C8, C9: footprint tscircuit:capacitor_cap0603 -> capacitor_cap0603
- C11: footprint tscircuit:capacitor_cap1206 -> capacitor_cap1206; moved to B.Cu
- C15, C16, C17: footprint tscircuit:capacitor_cap0805 -> capacitor_cap0805; moved to B.Cu
- C21, C47, C5, C62: footprint tscircuit:capacitor_cap1206 -> capacitor_cap1206
- C22, C23: footprint tscircuit:EEUFR1J471 -> EEUFR1J471
- C25, C27, C30, C32, C33, C34, C35, C66, C67, C68: footprint tscircuit:capacitor_cap0805 -> capacitor_cap0805
- D1, D7: footprint tscircuit:BAV21W-7-F -> BAV21W-7-F
- D10, D4, D5, D6, D8, D9: footprint tscircuit:BAV21W-7-F -> BAV21W-7-F; moved to B.Cu
- D11: footprint tscircuit:SS110 -> SS110; moved to B.Cu
- D12: footprint tscircuit:SS110 -> SS110
- D2: footprint tscircuit:SM24CANB-02HTG -> SM24CANB-02HTG
- D3: footprint tscircuit:PSM712-LF-T7 -> PSM712-LF-T7
- J1: footprint tscircuit:USB4105-GF-A -> USB4105-GF-A
- J2: footprint tscircuit:B4P-VH_LF_SN -> B4P-VH_LF_SN
- J3: footprint tscircuit:B2P-VH_LF_SN -> B2P-VH_LF_SN
- J6: footprint tscircuit:B8B-PH-K-S_LF_SN -> B8B-PH-K-S_LF_SN
- J7: footprint tscircuit:B6B-PH-K-S_LF_SN -> B8B-PH-K-S_LF_SN
- J9: footprint tscircuit:B4B-PH-K-S_LF_SN -> B4B-PH-K-S_LF_SN
- L1: footprint tscircuit:SWPA6045S220MT -> SWPA6045S220MT; moved to B.Cu
- L2: footprint tscircuit:SWPA6045S220MT -> SWPA6045S220MT
- Q1: value BSS123LT1G -> Q1; footprint tscircuit:BSS123LT1G -> BSS123LT1G
- Q10: value CSD19534Q5A -> Q10; footprint tscircuit:CSD19534Q5A -> CSD19534Q5A
- Q11: value CSD19534Q5A -> Q11; footprint tscircuit:CSD19534Q5A -> CSD19534Q5A
- Q12: value CSD19534Q5A -> Q12; footprint tscircuit:CSD19534Q5A -> CSD19534Q5A
- Q13: value CSD19534Q5A -> Q13; footprint tscircuit:CSD19534Q5A -> CSD19534Q5A
- Q14: value MMBT5551LT1G -> Q14; footprint tscircuit:MMBT5551LT1G -> MMBT5551LT1G
- Q15: value MMBT5551LT1G -> Q15; footprint tscircuit:MMBT5551LT1G -> MMBT5551LT1G
- Q16: value CSD19534Q5A -> Q16; footprint tscircuit:CSD19534Q5A -> CSD19534Q5A
- Q17: value MMBT5551LT1G -> Q17; footprint tscircuit:MMBT5551LT1G -> MMBT5551LT1G
- Q18: value MMBT5551LT1G -> Q18; footprint tscircuit:MMBT5551LT1G -> MMBT5551LT1G
- Q19: value MMBT5551LT1G -> Q19; footprint tscircuit:MMBT5551LT1G -> MMBT5551LT1G
- Q2: value MMBT5551LT1G -> Q2; footprint tscircuit:MMBT5551LT1G -> MMBT5551LT1G
- Q20: value MMBT5551LT1G -> Q20; footprint tscircuit:MMBT5551LT1G -> MMBT5551LT1G
- Q21: value MMBT5551LT1G -> Q21; footprint tscircuit:MMBT5551LT1G -> MMBT5551LT1G
- Q22: value MMBT5551LT1G -> Q22; footprint tscircuit:MMBT5551LT1G -> MMBT5551LT1G
- Q23: value MMBT5551LT1G -> Q23; footprint tscircuit:MMBT5551LT1G -> MMBT5551LT1G
- Q24: value MMBT5551LT1G -> Q24; footprint tscircuit:MMBT5551LT1G -> MMBT5551LT1G; moved to B.Cu
- Q25: value MMBT5551LT1G -> Q25; footprint tscircuit:MMBT5551LT1G -> MMBT5551LT1G; moved to B.Cu
- Q3: value MMBT5551LT1G -> Q3; footprint tscircuit:MMBT5551LT1G -> MMBT5551LT1G
- Q4: value CSD19534Q5A -> Q4; footprint tscircuit:CSD19534Q5A -> CSD19534Q5A
- Q5: value BSS123LT1G -> Q5; footprint tscircuit:BSS123LT1G -> BSS123LT1G
- Q6: value CSD19534Q5A -> Q6; footprint tscircuit:CSD19534Q5A -> CSD19534Q5A
- Q7: value CSD19534Q5A -> Q7; footprint tscircuit:CSD19534Q5A -> CSD19534Q5A
- Q8: value CSD19534Q5A -> Q8; footprint tscircuit:CSD19534Q5A -> CSD19534Q5A
- Q9: value CSD19534Q5A -> Q9; footprint tscircuit:CSD19534Q5A -> CSD19534Q5A
- R1, R100, R101, R11, R16, R17, R18, R2, R7, R74, R91, R92, R93, R94, R95, R96, R98, R99: footprint tscircuit:resistor_res0603 -> resistor_res0603; moved to B.Cu
- R10, R102, R103, R104, R12, R13, R14, R15, R19, R20, R21, R22, R23, R24, R25, R26, R27, R28, R29, R3, R30, R31, R32, R33, R34, R35, R36, R37, R38, R39, R4, R40, R41, R42, R43, R44, R45, R46, R47, R48, R49, R5, R50, R51, R52, R53, R54, R55, R56, R57, R58, R59, R6, R60, R61, R62, R63, R64, R65, R66, R67, R68, R69, R70, R71, R72, R73, R75, R76, R77, R78, R79, R8, R80, R81, R82, R83, R84, R85, R86, R87, R88, R89, R9, R90, R97: footprint tscircuit:resistor_res0603 -> resistor_res0603
- SW1: footprint tscircuit:TS-1088-AR02016 -> TS-1088-AR02016; moved to B.Cu
- U1: footprint tscircuit:TPD4S480RUKR -> TPD4S480RUKR
- U10, U11, U4: footprint tscircuit:SN74LVC1G08DBVR -> SN74LVC1G08DBVR
- U12: footprint tscircuit:TL431AIDBZR -> TL431AIDBZR
- U13, U14: footprint tscircuit:TLV3201AIDBVR -> TLV3201AIDBVR
- U15: footprint tscircuit:UCC27511DBVR -> UCC27511DBVR
- U16: footprint tscircuit:STM32G0B1CBT6 -> STM32G0B1CBT6
- U17: footprint tscircuit:W25Q32JVSSIQ -> W25Q32JVSSIQ
- U18: footprint tscircuit:AS5047P-ATSM -> AS5047P-ATSM; moved to B.Cu
- U19: footprint tscircuit:TCAN332DR -> TCAN332DR
- U2: footprint tscircuit:TPS26750SRSMR -> TPS26750SRSMR
- U20: footprint tscircuit:MAX3485EESA_T -> MAX3485EESA_T
- U21: footprint tscircuit:MAX3232ESE_T -> MAX3232ESE_T
- U22: footprint tscircuit:LMR36510ADDAR -> LMR36510ADDAR
- U23, U24: footprint tscircuit:LM66100DCKR -> LM66100DCKR
- U3: footprint tscircuit:M24512-RMN6TP -> M24512-RMN6TP
- U5: footprint tscircuit:LMR36510ADDAR -> LMR36510ADDAR; moved to B.Cu
- U6: footprint tscircuit:TPS26631RGER -> TPS26631RGER
- U7: footprint tscircuit:TMC5160A-TA-T -> TMC5160A-TA-T
- U8, U9: footprint tscircuit:74LVC1G157GW_125 -> 74LVC1G157GW_125
- Y1: footprint tscircuit:X322516MLB4SI -> X322516MLB4SI
- moved J2 74.4 mm to (120.0, 139.0)
- moved R95 39.3 mm to (134.0, 97.0), turned to 180 degrees
- moved R101 26.2 mm to (130.0, 128.5)
- moved R100 26.0 mm to (127.0, 127.0)
- moved D8 24.5 mm to (138.0, 109.0)
- moved R98 24.3 mm to (118.0, 127.0)
- moved R99 24.2 mm to (122.0, 131.0)
- moved Q1 23.8 mm to (76.0, 59.5)
- moved R94 23.3 mm to (134.0, 100.0)
- moved D4 22.9 mm to (96.0, 124.0)
- moved R93 22.3 mm to (134.0, 103.0)
- moved SW1 22.0 mm to (88.0, 120.0), turned to 180 degrees
- moved R96 21.7 mm to (130.0, 118.0)
- moved D5 21.3 mm to (104.0, 124.0)
- moved R91 21.0 mm to (134.0, 112.0)
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Connections:
- J1 pad 11: USB_DP_CONN -> (no net)
- J1 pad 12: USB_DM_CONN -> (no net)
- J1 pad 13: USB_DP_CONN -> (no net)
- J1 pad 14: USB_DM_CONN -> (no net)
- J7 pad 1: DIN0_24V -> HOME_24V
- J7 pad 2: DIN1_24V -> STOPL_24V
- J7 pad 3: STOPL_24V -> STOPR_24V
- J7 pad 4: STOPR_24V -> DIN0_24V
- J7 pad 5: HOME_24V -> DIN1_24V
- J7 pad 6: GND -> STEP_24V
- U16 pad 19: (no net) -> USB_DATA_VBUS_SENSE
Routing:
- net GND: track 209.0 -> 989.8 mm, vias 152 -> 14
- net V3V3: track 416.0 -> 473.0 mm, vias 13 -> 12
- net VMOTOR: track 334.5 -> 385.6 mm, vias 44 -> 42
- net STEP_24V: track 24.4 -> 70.9 mm, vias 1 -> 3
- net DIR_24V: track 23.6 -> 68.2 mm, vias 0 -> 1
- net USB_VBUS: track 88.8 -> 128.9 mm, vias 11 -> 28
- net USB_DATA_VBUS_SENSE: track 0.00 -> 38.9 mm, vias 0 -> 2
- net HOME_IN: track 67.6 -> 96.9 mm, vias 3 -> 4
- net OUT1_BASE: track 36.0 -> 11.7 mm, vias 2 -> 0
- net USB_DATA_VBUS: track 0.00 -> 24.0 mm
- net CC_FAULT_N: track 5.05 -> 29.0 mm, vias 3 -> 4
- net OUT0_DRIVE: track 82.2 -> 58.2 mm
- net NRST: track 48.2 -> 25.4 mm, vias 3 -> 1
- net HOME_IN_BASE: track 27.5 -> 49.6 mm
- net OUT0_BASE: track 34.4 -> 12.5 mm, vias 3 -> 0
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- added copper zone on B.Cu, net MOTOR_A1
- added copper zone on B.Cu, net MOTOR_A2
- added copper zone on B.Cu, net MOTOR_B2
- added copper zone on In1.Cu, net SENSE_B
- added copper zone on In2.Cu, net SENSE_B
- added copper zone on In1.Cu, net USB_VBUS
- added copper zone on In2.Cu, net USB_VBUS
- added copper zone on B.Cu, net VMOTOR
- removed copper zone on In1.Cu, net BRAKE_RETURN
- removed copper zone on In2.Cu, net BRAKE_RETURN
- removed copper zone on B.Cu, net CC_FAULT_N
- removed copper zone on F.Cu, net CC_FAULT_N
- removed copper zone on In2.Cu, net EFUSE_IN
- removed copper zone on B.Cu, net GND
- removed copper zone on F.Cu, net GND
- removed copper zone on In2.Cu, net MOTOR_A1
- removed copper zone on F.Cu, net V3V3
Other:
- outline, holes or cut-outs redrawn
- board text added: "ENC TEST"
- board text added: "J10 USB DATA"
- board text added: "J2 MOTOR"
- board text added: "SWD TEST"
- board text added: "U18 ENCODER"
- board text removed: "J1"
- board text removed: "J2"
- board text removed: "J4"
- board text removed: "J5"
- board text removed: "J8"
- board text removed: "Q1"
- board text removed: "Q10"
- board text removed: "Q11"
- board text removed: "Q12"
- board text removed: "Q13"
- board text removed: "Q14"
- board text removed: "Q15"
- board text removed: "Q16"
- board text removed: "Q17"
- board text removed: "Q18"
- board text removed: "Q19"
- board text removed: "Q2"
- board text removed: "Q20"
- board text removed: "Q21"
- board text removed: "Q22"
- board text removed: "Q23"
- board text removed: "Q24"
- board text removed: "Q25"
- board text removed: "Q3"
- board text removed: "Q4"
- board text removed: "Q5"
- board text removed: "Q6"
- board text removed: "Q7"
- board text removed: "Q8"
- board text removed: "Q9"
- board text removed: "RS1"
- board text removed: "RS2"
- board text removed: "SW1"
- board text removed: "U1"
- board text removed: "U18"
- board text removed: "U19"
- board text removed: "U21"
- board text removed: "U5"
- board text removed: "ts"
