File: dist/manufacturing/kicad-project/index.kicad_sch (KiCad schematic)
At the start: 0 parts

Commit message: Complete orderable PD1180-EPR board release
Other:
- removed sheet USB-C EPR and USB Data
- added sheet USB-C EPR Power and USB Data (usb_pd.kicad_sch)
Changed lines of the file:
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@@
       (color 0 0 0 0)
     )
-    (property "Sheetname" "USB-C EPR and USB Data"
+    (property "Sheetname" "USB-C EPR Power and USB Data"
       (id 0)
       (at 25.4 24.7 0)
@@
     (instances
       (project ""
-        (path "/64ba309c-a36f-4940-acc6-e52d2d121bae"
+        (path "/f5f6ca0d-0209-4855-99b3-5a1edaa43ca4"
           (page "2")
         )
@@
     (instances
       (project ""
-        (path "/64ba309c-a36f-4940-acc6-e52d2d121bae"
+        (path "/f5f6ca0d-0209-4855-99b3-5a1edaa43ca4"
           (page "3")
         )
@@
     (instances
       (project ""
-        (path "/64ba309c-a36f-4940-acc6-e52d2d121bae"
+        (path "/f5f6ca0d-0209-4855-99b3-5a1edaa43ca4"
           (page "4")
         )
@@
     (instances
       (project ""
-        (path "/64ba309c-a36f-4940-acc6-e52d2d121bae"
+        (path "/f5f6ca0d-0209-4855-99b3-5a1edaa43ca4"
           (page "5")
         )
@@
     (instances
       (project ""
-        (path "/64ba309c-a36f-4940-acc6-e52d2d121bae"
+        (path "/f5f6ca0d-0209-4855-99b3-5a1edaa43ca4"
           (page "6")
         )
@@
     (instances
       (project ""
-        (path "/64ba309c-a36f-4940-acc6-e52d2d121bae"
+        (path "/f5f6ca0d-0209-4855-99b3-5a1edaa43ca4"
           (page "7")
         )
@@
     (instances
       (project ""
-        (path "/64ba309c-a36f-4940-acc6-e52d2d121bae"
+        (path "/f5f6ca0d-0209-4855-99b3-5a1edaa43ca4"
           (page "8")
         )
@@
     (instances
       (project ""
-        (path "/64ba309c-a36f-4940-acc6-e52d2d121bae"
+        (path "/f5f6ca0d-0209-4855-99b3-5a1edaa43ca4"
           (page "9")
         )
@@
     (instances
       (project ""
-        (path "/64ba309c-a36f-4940-acc6-e52d2d121bae"
+        (path "/f5f6ca0d-0209-4855-99b3-5a1edaa43ca4"
           (page "10")
         )
@@
     (instances
       (project ""
-        (path "/64ba309c-a36f-4940-acc6-e52d2d121bae"
+        (path "/f5f6ca0d-0209-4855-99b3-5a1edaa43ca4"
           (page "11")
         )
@@
     (instances
       (project ""
-        (path "/64ba309c-a36f-4940-acc6-e52d2d121bae"
+        (path "/f5f6ca0d-0209-4855-99b3-5a1edaa43ca4"
           (page "12")
         )
@@
     (instances
       (project ""
-        (path "/64ba309c-a36f-4940-acc6-e52d2d121bae"
+        (path "/f5f6ca0d-0209-4855-99b3-5a1edaa43ca4"
           (page "13")
         )
