File: dist/manufacturing/kicad-project/inputs.kicad_sch (KiCad schematic)
At the start: 68 parts, among them J7 B6B-PH-K-S(LF)(SN), J8 B4B-PH-K-S(LF)(SN), Q17 MMBT5551LT1G, Q18 MMBT5551LT1G, Q19 MMBT5551LT1G, Q20 MMBT5551LT1G, Q21 MMBT5551LT1G, Q22 MMBT5551LT1G, Q23 MMBT5551LT1G

Commit message: Complete orderable PD1180-EPR board release
Parts:
- removed GND (x23): GND, symbol Custom:rail_down
- removed J7: B6B-PH-K-S(LF)(SN), symbol Device:J_B6B-PH-K-S_LF_SN
- removed J8: B4B-PH-K-S(LF)(SN), symbol Device:J_B4B-PH-K-S_LF_SN
- removed Q17, Q18, Q19, Q20, Q21, Q22, Q23: MMBT5551LT1G, symbol Device:U_MMBT5551LT1G
- removed V3V3 (x8): V3V3, symbol Custom:rail_up
- added GND (x22): GND, symbol Custom:rail_down
- added J7: B8B-PH-K-S(LF)(SN), symbol Device:J_B8B-PH-K-S_LF_SN
- added Q17: Q17, symbol Custom:MMBT5551LT1G_NPN
- added Q18: Q18, symbol Custom:MMBT5551LT1G_NPN
- added Q19: Q19, symbol Custom:MMBT5551LT1G_NPN
- added Q20: Q20, symbol Custom:MMBT5551LT1G_NPN
- added Q21: Q21, symbol Custom:MMBT5551LT1G_NPN
- added Q22: Q22, symbol Custom:MMBT5551LT1G_NPN
- added Q23: Q23, symbol Custom:MMBT5551LT1G_NPN
- added V3V3 (x7): V3V3, symbol Custom:rail_up
Connections:
- net at R88.1: now also V3V3.1
- net at R85.1: now also V3V3.1
- net at R87.2: now also GND.1
- net at D10.2 (1): now also GND.1
- net at R86.2: now also Q20.1 (base)
- net at R77.2: now also Q17.1 (base)
- net at R89.2: now also Q21.1 (base)
- net at D4.2 (1): now also GND.1
- net at R78.2: now also GND.1
- net at D7.2 (1): now also GND.1
- net at D6.2 (1): now also GND.1
- net at R84.2: now also GND.1
- net at R90.2: now also GND.1
- net at R97.1: now also V3V3.1
- net at R91.1: now also V3V3.1
- net at R95.2: now also Q23.1 (base)
- net at D9.2 (1): now also GND.1
- net at R80.2: now also Q18.1 (base)
- net at R96.2: now also GND.1
- net at R83.2: now also Q19.1 (base)
- net at R79.1: now also V3V3.1
- net at D8.2 (1): now also GND.1
- net at R93.2: now also GND.1
- net at R82.1: now also V3V3.1
- net at R92.2: now also Q22.1 (base)
- net at R81.2: now also GND.1
- net at D5.2 (1): now also GND.1
- net at R94.1: now also V3V3.1
- new net: GND.1, Q20.2 (emitter)
- new net: GND.1, Q18.2 (emitter)
- new net: GND.1, J7.8
- new net: GND.1, Q22.2 (emitter)
- new net: GND.1, Q17.2 (emitter)
- new net: GND.1, Q19.2 (emitter)
- new net: GND.1, Q21.2 (emitter)
- new net: GND.1, Q23.2 (emitter)
Other:
- note added: "Non-isolated 24 V inputs. J7 consolidates home, stops, digital inputs and Step/Direction."
- note added: "Q17-Q23: 24 V tolerant NPN input conditioners for HOME, limits, DIN0/1 and Step/Direction signals."
- note removed: "Non-isolated 24 V inputs. J8 is Step/Direction; J7 is home, stop and digital inputs."

Commit message: Fix schematic style and top-side reset switch
Parts:
- removed GND (x22): GND, symbol Custom:rail_down
- removed V3V3 (x7): V3V3, symbol Custom:rail_up
- added GND (x22): GND, symbol Custom:rail_down
- added V3V3 (x7): V3V3, symbol Custom:rail_up
Connections:
- net at Q20.2 (E): now also GND.1
- net at Q18.2 (E): now also GND.1
- net at R94.1: now also V3V3.1
- net at R85.1: now also V3V3.1
- net at D8.2 (1): now also GND.1
- net at R82.1: now also V3V3.1
- net at R81.2: now also GND.1
- net at J7.8: now also GND.1
- net at D5.2 (1): now also GND.1
- net at R84.2: now also GND.1
- net at D10.2 (1): now also GND.1
- net at R97.1: now also V3V3.1
- net at R79.1: now also V3V3.1
- net at D7.2 (1): now also GND.1
- net at Q22.2 (E): now also GND.1
- net at Q17.2 (E): now also GND.1
- net at R88.1: now also V3V3.1
- net at R96.2: now also GND.1
- net at D6.2 (1): now also GND.1
- net at Q19.2 (E): now also GND.1
- net at Q21.2 (E): now also GND.1
- net at R87.2: now also GND.1
- net at R91.1: now also V3V3.1
- net at Q23.2 (E): now also GND.1
- net at D4.2 (1): now also GND.1
- net at R93.2: now also GND.1
- net at R90.2: now also GND.1
- net at R78.2: now also GND.1
- net at D9.2 (1): now also GND.1
- net DIR_IN_BASE: no longer names the net of D10.1 (2)
- net HOME_IN_BASE: no longer names the net of D8.1 (2)
- net STEP_IN_BASE: no longer names the net of D9.1 (2)
- net STOP_L_BASE: no longer names the net of D6.1 (2)
- net STOP_R_BASE: no longer names the net of D7.1 (2)

Commit message: Use one USB-C port for PD and data
Parts:
- removed GND (x22): GND, symbol Custom:rail_down
- removed V3V3 (x7): V3V3, symbol Custom:rail_up
- added GND (x22): GND, symbol Custom:rail_down
- added V3V3 (x7): V3V3, symbol Custom:rail_up
Connections:
- net at R91.1: now also V3V3.1
- net at R85.1: now also V3V3.1
- net at R97.1: now also V3V3.1
- net at Q22.2 (E): now also GND.1
- net at R79.1: now also V3V3.1
- net at R94.1: now also V3V3.1
- net at Q23.2 (E): now also GND.1
- net at R82.1: now also V3V3.1
- net at Q20.2 (E): now also GND.1
- net at Q19.2 (E): now also GND.1
- net at R87.2: now also GND.1
- net at D6.2 (1): now also GND.1
- net at D9.2 (1): now also GND.1
- net at Q21.2 (E): now also GND.1
- net at R93.2: now also GND.1
- net at R96.2: now also GND.1
- net at Q17.2 (E): now also GND.1
- net at R78.2: now also GND.1
- net at Q18.2 (E): now also GND.1
- net at J7.8: now also GND.1
- net at R81.2: now also GND.1
- net at D8.2 (1): now also GND.1
- net at R88.1: now also V3V3.1
- net at R84.2: now also GND.1
- net at D4.2 (1): now also GND.1
- net at D5.2 (1): now also GND.1
- net at D7.2 (1): now also GND.1
- net at R90.2: now also GND.1
- net at D10.2 (1): now also GND.1

Commit message: fix: finalize single-port EPR controller
Parts:
- removed GND (x22): GND, symbol Custom:rail_down
- removed V3V3 (x7): V3V3, symbol Custom:rail_up
- D10, D4, D5, D6, D7, D8, D9: value BAV21W-7-F -> D; footprint (none) -> BAV21W-7-F
- J7: value B8B-PH-K-S(LF)(SN) -> J7; footprint (none) -> B8B-PH-K-S_LF_SN
- Q17, Q18, Q19, Q20, Q21, Q22, Q23: footprint (none) -> MMBT5551LT1G
- R77, R78, R79, R80, R81, R82, R83, R84, R85, R86, R87, R88, R89, R90, R91, R92, R93, R94, R95, R96, R97: footprint (none) -> resistor_res0603
Connections:
- net DIN1_BASE: now reaches R81.1
- net DIN1_BASE: now also D5.1 (2), Q18.1 (B), R80.2
- net GND: now reaches R81.2
- net GND: now also D10.2 (1), D4.2 (1), D5.2 (1), D6.2 (1), D7.2 (1), D8.2 (1), D9.2 (1), J7.8, Q17.2 (E), Q18.2 (E), Q19.2 (E), Q20.2 (E), Q21.2 (E), Q22.2 (E), Q23.2 (E), R78.2, R84.2, R87.2, R90.2, R93.2, R96.2
- net DIR_24V: now reaches R95.1
- net DIR_24V: now also J7.7
- net DIR_IN_BASE: now reaches Q23.1 (B), R95.2
- net DIR_IN_BASE: now also D10.1 (2), R96.1
- net HOME_IN_BASE: now reaches Q21.1 (B), R89.2
- net HOME_IN_BASE: now also D8.1 (2), R90.1
- net HOME_IN: now reaches Q21.3 (C)
- net HOME_IN: now also R91.2
- net V3V3: now reaches R97.1
- net V3V3: now also R79.1, R82.1, R85.1, R88.1, R91.1, R94.1
- net DIR_IN: now reaches R97.2
- net DIR_IN: now also Q23.3 (C)
- net STOP_R_BASE: now reaches D7.1 (2)
- net STOP_R_BASE: now also Q20.1 (B), R86.2, R87.1
- net STOP_L: now reaches R85.2
- net STOP_L: now also Q19.3 (C)
- net STEP_24V: now reaches R92.1
- net STEP_24V: now also J7.6
- net STEP_IN_BASE: now reaches Q22.1 (B), R92.2
- net STEP_IN_BASE: now also D9.1 (2), R93.1
- net STOPR_24V: now reaches R86.1
- net STOPR_24V: now also J7.3
- net DIN0_BASE: now reaches R78.1
- net DIN0_BASE: now also D4.1 (2), Q17.1 (B), R77.2
- net STOP_L_BASE: now reaches R84.1
- net STOP_L_BASE: now also D6.1 (2), Q19.1 (B), R83.2
- net DIN0: now reaches R79.2
- net DIN0: now also Q17.3 (C)
- net HOME_24V: now reaches J7.1
- net HOME_24V: now also R89.1
- net STOPL_24V: now reaches J7.2
- net STOPL_24V: now also R83.1
- net DIN0_24V: now reaches J7.4
- net DIN0_24V: now also R77.1
- net DIN1_24V: now reaches J7.5
- net DIN1_24V: now also R80.1
- net STOP_R: now reaches R88.2
- net STOP_R: now also Q20.3 (C)
- net DIN1: now reaches Q18.3 (C)
- net DIN1: now also R82.2
- net STEP_IN: now reaches Q22.3 (C)
- net STEP_IN: now also R94.2

Commit message: Implement dual USB power/data ECO and consolidate industrial I/O
Parts:
- removed J7: J7, B8B-PH-K-S_LF_SN, symbol Device:J_B8B-PH-K-S_LF_SN
- removed Q17: Q17, MMBT5551LT1G, symbol Custom:MMBT5551LT1G_NPN
- removed Q18: Q18, MMBT5551LT1G, symbol Custom:MMBT5551LT1G_NPN
- removed Q19: Q19, MMBT5551LT1G, symbol Custom:MMBT5551LT1G_NPN
- removed Q20: Q20, MMBT5551LT1G, symbol Custom:MMBT5551LT1G_NPN
- removed Q21: Q21, MMBT5551LT1G, symbol Custom:MMBT5551LT1G_NPN
- removed Q22: Q22, MMBT5551LT1G, symbol Custom:MMBT5551LT1G_NPN
- removed Q23: Q23, MMBT5551LT1G, symbol Custom:MMBT5551LT1G_NPN
- added J7: B20B-PHDSS(LF)(SN), B20B-PHDSS_LF_SN, symbol Device:U_B20B-PHDSS_LF_SN
- added Q17: Q17, MMBT5551LT1G, symbol Custom:MMBT5551LT1G
- added Q18: Q18, MMBT5551LT1G, symbol Custom:MMBT5551LT1G
- added Q19: Q19, MMBT5551LT1G, symbol Custom:MMBT5551LT1G
- added Q20: Q20, MMBT5551LT1G, symbol Custom:MMBT5551LT1G
- added Q21: Q21, MMBT5551LT1G, symbol Custom:MMBT5551LT1G
- added Q22: Q22, MMBT5551LT1G, symbol Custom:MMBT5551LT1G
- added Q23: Q23, MMBT5551LT1G, symbol Custom:MMBT5551LT1G
Connections:
- net DIN0: now also Q17.3 (C)
- net DIN0_24V: now also J7.4
- net DIN0_BASE: now also Q17.1 (B)
- net DIN1: now also Q18.3 (C)
- net DIN1_24V: now also J7.5
- net DIN1_BASE: now also Q18.1 (B)
- net DIR_24V: now also J7.7
- net DIR_IN: now also Q23.3 (C)
- net DIR_IN_BASE: now also Q23.1 (B)
- net GND: now also J7.11, J7.14, J7.8, Q17.2 (E), Q18.2 (E), Q19.2 (E), Q20.2 (E), Q21.2 (E), Q22.2 (E), Q23.2 (E)
- net HOME_24V: now also J7.1
- net HOME_IN: now also Q21.3 (C)
- net HOME_IN_BASE: now also Q21.1 (B)
- net STEP_24V: now also J7.6
- net STEP_IN: now also Q22.3 (C)
- net STEP_IN_BASE: now also Q22.1 (B)
- net STOPL_24V: now also J7.2
- net STOPR_24V: now also J7.3
- net STOP_L: now also Q19.3 (C)
- net STOP_L_BASE: now also Q19.1 (B)
- net STOP_R: now also Q20.3 (C)
- net STOP_R_BASE: now also Q20.1 (B)
- new net CAN_H: J7.12
- new net CAN_L: J7.13
- new net HW_ENABLE_24V: J7.18
- new net OUT0: J7.19
- new net OUT1: J7.20
- new net RS232_RX_CONN: J7.10
- new net RS232_TX_CONN: J7.9
- new net RS485_A: J7.15
- new net RS485_B: J7.16
- new net VMOTOR: J7.17
Other:
- note added: "CAN_H"
- note added: "CAN_L"
- note added: "HW_ENABLE_24V"
- note added: "Non-isolated 24 V inputs. J7: keyed 20-pin harness combines all control I/O and industrial buses; pinout is in hardware-contract.json."
- note added: "OUT0"
- note added: "OUT1"
- note added: "Q17-Q23: HOME, limits, DIN0/1 and Step/Direction conditioners. Q14: hardware enable on the motion sheet."
- note added: "RS232_RX_CONN"
- note added: "RS232_TX_CONN"
- note added: "RS485_A"
- note added: "RS485_B"
- note removed: "Non-isolated 24 V inputs. J7 consolidates home, stops, digital inputs and Step/Direction."
- note removed: "Q17-Q23: 24 V tolerant NPN input conditioners for HOME, limits, DIN0/1 and Step/Direction signals."
