File: dist/manufacturing/kicad-project/inputs.kicad_sch (KiCad schematic)
At the start: 36 parts, among them J7 B20B-PHDSS(LF)(SN), Q17 Q17, Q18 Q18, Q19 Q19, Q20 Q20, Q21 Q21, Q22 Q22, Q23 Q23

Commit message: Fix source warnings and organize schematic on A4 sheets
Parts:
- removed D10, D8, D9: D, BAV21W-7-F, symbol Device:diode_up
- removed J7: B20B-PHDSS(LF)(SN), B20B-PHDSS_LF_SN, symbol Device:U_B20B-PHDSS_LF_SN
- removed Q21: Q21, MMBT5551LT1G, symbol Custom:MMBT5551LT1G
- removed Q22: Q22, MMBT5551LT1G, symbol Custom:MMBT5551LT1G
- removed Q23: Q23, MMBT5551LT1G, symbol Custom:MMBT5551LT1G
- removed R89, R92, R95: 47kΩ, resistor_res0603, symbol Device:boxresistor_right
- removed R90, R93, R96: 10kΩ, resistor_res0603, symbol Device:boxresistor_down
- removed R91, R94, R97: 4.7kΩ, resistor_res0603, symbol Device:boxresistor_down
- Q17: value Q17 -> MMBT5551LT1G
- Q18: value Q18 -> MMBT5551LT1G
- Q19: value Q19 -> MMBT5551LT1G
- Q20: value Q20 -> MMBT5551LT1G
Other:
- note added: "16 / Home Limits and Digital Input 0"
- note added: "Non-isolated 24 V HOME, left/right STOP and DIN0 conditioning."
- note added: "The consolidated J7 harness is shown on the Step Direction and Industrial Harness sheet."
- note removed: "11 / 24 V Inputs and Step/Direction"
- note removed: "CAN_H"
- note removed: "CAN_L"
- note removed: "DIR_24V"
- note removed: "DIR_IN"
- note removed: "DIR_IN_BASE"
- note removed: "HOME_24V"
- note removed: "HOME_IN"
- note removed: "HOME_IN_BASE"
- note removed: "HW_ENABLE_24V"
- note removed: "Non-isolated 24 V inputs. J7: keyed 20-pin harness combines all control I/O and industrial buses; pinout is in hardware-contract.json."
- note removed: "OUT0"
- note removed: "OUT1"
- note removed: "Q17-Q23: HOME, limits, DIN0/1 and Step/Direction conditioners. Q14: hardware enable on the motion sheet."
- note removed: "RS232_RX_CONN"
- note removed: "RS232_TX_CONN"
- note removed: "RS485_A"
- note removed: "RS485_B"
- note removed: "STEP_24V"
- note removed: "STEP_IN"
- note removed: "STEP_IN_BASE"
