File: dist/manufacturing/kicad-project/motion.kicad_sch (KiCad schematic)
At the start: 66 parts, among them Q14 MMBT5551LT1G, Q15 MMBT5551LT1G, U10 SN74LVC1G08DBVR, U11 SN74LVC1G08DBVR, U7 TMC5160A-TA-T, U8 74LVC1G157GW,125, U9 74LVC1G157GW,125

Commit message: Complete orderable PD1180-EPR board release
Parts:
- removed C31: 100nF, symbol Device:capacitor_right
- removed C35: 220nF, symbol Device:capacitor_right
- removed GND (x16): GND, symbol Custom:rail_down
- removed Q14, Q15: MMBT5551LT1G, symbol Device:U_MMBT5551LT1G
- removed TMC_12V (x2): TMC_12V, symbol Custom:rail_up
- removed TMC_5V (x2): TMC_5V, symbol Custom:rail_up
- removed TMC_VCC (x2): TMC_VCC, symbol Custom:rail_up
- removed V3V3 (x6): V3V3, symbol Custom:rail_up
- removed VMOTOR (x5): VMOTOR, symbol Custom:rail_up
- added C31: 100nF, symbol Device:capacitor_up
- added C35: 220nF, symbol Device:capacitor_down
- added GND (x21): GND, symbol Custom:rail_down
- added Q14: Q14, symbol Custom:MMBT5551LT1G_NPN
- added Q15: Q15, symbol Custom:MMBT5551LT1G_NPN
- added TMC_12V (x2): TMC_12V, symbol Custom:rail_up
- added TMC_5V (x2): TMC_5V, symbol Custom:rail_up
- added TMC_VCC (x2): TMC_VCC, symbol Custom:rail_up
- added V3V3 (x10): V3V3, symbol Custom:rail_up
- added VMOTOR (x4): VMOTOR, symbol Custom:rail_up
Connections:
- net ENABLE_CHAIN: now also Q15.3 (collector)
- net GND: no longer U7.30 (GNDD2), U7.49 (EP)
- net HW_ENABLE_BASE: no longer R58.1
- net at U11.3 (GND): now also R56.2, GND.1
- net at C36.2: now also GND.1
- net at C25.1: now also TMC_12V.1
- net at R35.1, R37.1: now also V3V3.1
- net at R34.2: now also TMC_VCC.1
- net at C29.1: now also VMOTOR.1
- net at C39.1: now also V3V3.1; no longer U11.5 (VCC)
- net at C39.2: now also GND.1
- net at C61.1: now also VMOTOR.1
- net at R34.1: now also TMC_5V.1
- net at C61.2: now also GND.1
- net at U8.2 (GND): now also GND.1
- net at C26.1, U7.5 (5VOUT): now also TMC_5V.1
- net at C25.2: now also GND.1; no longer C26.2
- net at R36.2: now also GND.1
- net at U9.5 (VCC): now also V3V3.1; no longer C37.1
- net at U9.2 (GND): now also GND.1
- net at U10.3 (GND): now also R54.2, GND.1
- net at U10.5 (VCC): now also V3V3.1; no longer C38.1
- net at C38.2: now also GND.1; no longer R54.2
- net at C28.1: now also V3V3.1
- net at C36.1: now also V3V3.1; no longer U8.5 (VCC)
- net at C37.2: now also GND.1
- net at R57.2: now also Q15.1 (base)
- net at U7.10 (SRBL), U7.11 (TST_MODE), U7.12 (CLK)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: now also GND.1
- net at D1.2 (1): now also GND.1
- net at U7.3 (12VOUT): now also TMC_12V.1
- net at U7.33 (VS): now also U7.4 (VSA), VMOTOR.1
- net at R58.2: now also GND.1
- net HW_ENABLE_24V: no longer names the net of R57.1
- net SD_MODE: no longer names the net of R36.1
- new net: C27.2, GND.1
- new net: C31.2, VMOTOR.1
- new net: U8.5 (VCC), V3V3.1
- new net: C26.2, GND.1
- new net: GND.1, U7.30 (GNDD2)
- new net: GND.1, U7.49 (EP)
- new net: C28.2, GND.1
- new net: C37.1, V3V3.1
- new net: C29.2, GND.1
- new net: U11.5 (VCC), V3V3.1
- new net: C38.1, V3V3.1
- new net: GND.1, Q15.2 (emitter)
- new net TMC_VCP: C31.1
Other:
- note added: "HW_ENABLE_24V"
- note added: "U7: motion controller and gate driver. U8/U9: Step/Dir limit multiplexers. U10/U11 + Q14/Q15: hardwired enable interlock."

Commit message: Fix schematic style and top-side reset switch
Parts:
- removed GND (x21): GND, symbol Custom:rail_down
- removed TMC_12V (x2): TMC_12V, symbol Custom:rail_up
- removed TMC_5V (x2): TMC_5V, symbol Custom:rail_up
- removed TMC_VCC (x2): TMC_VCC, symbol Custom:rail_up
- removed V3V3 (x10): V3V3, symbol Custom:rail_up
- removed VMOTOR (x4): VMOTOR, symbol Custom:rail_up
- added GND (x20): GND, symbol Custom:rail_down
- added TMC_12V (x2): TMC_12V, symbol Custom:rail_up
- added TMC_5V (x2): TMC_5V, symbol Custom:rail_up
- added TMC_VCC (x2): TMC_VCC, symbol Custom:rail_up
- added V3V3 (x9): V3V3, symbol Custom:rail_up
- added VMOTOR (x3): VMOTOR, symbol Custom:rail_up
Connections:
- net at C27.2: now also GND.1
- net at C28.1: now also V3V3.1
- net at C25.1: now also TMC_12V.1
- net at C25.2: now also GND.1
- net at R54.2, U10.3 (GND): now also GND.1
- net at U10.5 (VCC): now also V3V3.1
- net at C31.2: now also VMOTOR.1
- net at U8.2 (GND): now also GND.1
- net at C38.2: now also GND.1
- net at R34.1: now also TMC_5V.1
- net at R34.2: now also TMC_VCC.1
- net at C36.1: now also U8.5 (VCC), V3V3.1
- net at U9.5 (VCC): now also V3V3.1
- net at R58.2: now also GND.1
- net at C39.1: now also V3V3.1
- net at C39.2: now also GND.1
- net at C26.1, U7.5 (5VOUT): now also TMC_5V.1
- net at C26.2: now also GND.1
- net at U7.10 (SRBL), U7.11 (TST_MODE), U7.12 (CLK)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: now also GND.1
- net at U7.3 (12VOUT): now also TMC_12V.1
- net at U7.30 (GNDD2): now also GND.1
- net at U7.33 (VS), U7.4 (VSA): now also VMOTOR.1
- net at U7.49 (EP): now also GND.1
- net at C37.2: now also GND.1
- net at C36.2: now also GND.1
- net at C61.1: now also C29.1, VMOTOR.1
- net at C28.2: now also GND.1
- net at D1.2 (1): now also GND.1
- net at C37.1: now also V3V3.1
- net at C29.2: now also C61.2, GND.1
- net at U9.2 (GND): now also GND.1
- net at U11.5 (VCC): now also V3V3.1
- net at R56.2, U11.3 (GND): now also GND.1
- net at C38.1: now also V3V3.1
- net at Q15.2 (E): now also GND.1
- net at R36.2: now also GND.1
- net at R35.1, R37.1: now also V3V3.1

Commit message: Use one USB-C port for PD and data
Parts:
- removed GND (x20): GND, symbol Custom:rail_down
- removed TMC_12V (x2): TMC_12V, symbol Custom:rail_up
- removed TMC_5V (x2): TMC_5V, symbol Custom:rail_up
- removed TMC_VCC (x2): TMC_VCC, symbol Custom:rail_up
- removed V3V3 (x9): V3V3, symbol Custom:rail_up
- removed VMOTOR (x3): VMOTOR, symbol Custom:rail_up
- added GND (x20): GND, symbol Custom:rail_down
- added TMC_12V (x2): TMC_12V, symbol Custom:rail_up
- added TMC_5V (x2): TMC_5V, symbol Custom:rail_up
- added TMC_VCC (x2): TMC_VCC, symbol Custom:rail_up
- added V3V3 (x9): V3V3, symbol Custom:rail_up
- added VMOTOR (x3): VMOTOR, symbol Custom:rail_up
Connections:
- net at C29.2, C61.2: now also GND.1
- net at R58.2: now also GND.1
- net at C25.1: now also TMC_12V.1
- net at C25.2: now also GND.1
- net at R35.1, R37.1: now also V3V3.1
- net at U7.49 (EP): now also GND.1
- net at R56.2, U11.3 (GND): now also GND.1
- net at C28.2: now also GND.1
- net at R54.2, U10.3 (GND): now also GND.1
- net at U10.5 (VCC): now also V3V3.1
- net at C39.2: now also GND.1
- net at C26.1, U7.5 (5VOUT): now also TMC_5V.1
- net at R34.1: now also TMC_5V.1
- net at U8.2 (GND): now also GND.1
- net at C28.1: now also V3V3.1
- net at C37.2: now also GND.1
- net at C36.1, U8.5 (VCC): now also V3V3.1
- net at U11.5 (VCC): now also V3V3.1
- net at C38.1: now also V3V3.1
- net at C38.2: now also GND.1
- net at C29.1, C61.1: now also VMOTOR.1
- net at D1.2 (1): now also GND.1
- net at C37.1: now also V3V3.1
- net at Q15.2 (E): now also GND.1
- net at U7.10 (SRBL), U7.11 (TST_MODE), U7.12 (CLK)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: now also GND.1
- net at U7.3 (12VOUT): now also TMC_12V.1
- net at U7.30 (GNDD2): now also GND.1
- net at U7.33 (VS), U7.4 (VSA): now also VMOTOR.1
- net at C27.2: now also GND.1
- net at C31.2: now also VMOTOR.1
- net at U9.5 (VCC): now also V3V3.1
- net at C39.1: now also V3V3.1
- net at R36.2: now also GND.1
- net at U9.2 (GND): now also GND.1
- net at R34.2: now also TMC_VCC.1
- net at C36.2: now also GND.1
- net at C26.2: now also GND.1

Commit message: fix: finalize single-port EPR controller
Parts:
- removed GND (x20): GND, symbol Custom:rail_down
- removed TMC_12V (x2): TMC_12V, symbol Custom:rail_up
- removed TMC_5V (x2): TMC_5V, symbol Custom:rail_up
- removed TMC_VCC (x2): TMC_VCC, symbol Custom:rail_up
- removed V3V3 (x9): V3V3, symbol Custom:rail_up
- removed VMOTOR (x3): VMOTOR, symbol Custom:rail_up
- C25, C27, C30, C32, C33, C34, C35: footprint (none) -> capacitor_cap0805
- C26, C28, C29, C31, C36, C37, C38, C39, C61: footprint (none) -> capacitor_cap0603
- D1: value BAV21W-7-F -> D; footprint (none) -> BAV21W-7-F
- Q14, Q15: footprint (none) -> MMBT5551LT1G
- R34, R35, R36, R37, R54, R55, R56, R57, R58: footprint (none) -> resistor_res0603
- U10, U11: footprint (none) -> SN74LVC1G08DBVR
- U7: footprint (none) -> TMC5160A-TA-T
- U8, U9: footprint (none) -> 74LVC1G157GW_125
Connections:
- net ENABLE_CHAIN: now also Q14.2 (E)
- net GND: now also C25.2, C26.2, C27.2, C28.2, C29.2, C36.2, C37.2, C38.2, C39.2, C61.2, D1.2 (1), Q15.2 (E), R36.2, R54.2, R56.2, R58.2, U10.3 (GND), U11.3 (GND), U7.10 (SRBL), U7.11 (TST_MODE), U7.12 (CLK), U7.30 (GNDD2), U7.49 (EP), U7.6 (GNDA), U7.7 (SRAL), U8.2 (GND), U9.2 (GND)
- net HW_ENABLE_BASE: now also Q15.1 (B), R57.2, R58.1
- net TMC_VCP: now also U7.34 (VCP)
- net V3V3: now also C28.1, C36.1, C37.1, C38.1, C39.1, R35.1, R37.1, U10.5 (VCC), U11.5 (VCC), U8.5 (VCC), U9.5 (VCC)
- net MCU_RUN: now reaches U10.1 (A)
- net MCU_RUN: now also R54.1
- net MOTOR_PG: now reaches U10.2 (B)
- net RUN_PG: now reaches U10.4 (Y)
- net RUN_PG: now also U11.1 (A)
- net TMC_VCC: now reaches C27.1, U7.29 (VCC)
- net TMC_VCC: now also R34.2
- net BOOT_B1: now reaches C34.1
- net BOOT_B1: now also U7.2 (CB1)
- net MOTOR_B1: now reaches C34.2
- net MOTOR_B1: now also U7.48 (BMB1)
- net BOOT_B2: now reaches C35.1
- net BOOT_B2: now also U7.43 (CB2)
- net MOTOR_B2: now reaches C35.2
- net MOTOR_B2: now also U7.45 (BMB2)
- net VMOTOR: now reaches C31.2
- net VMOTOR: now also C29.1, C61.1, U7.33 (VS), U7.4 (VSA)
- net TMC_CS_N: now reaches R35.2
- net TMC_CS_N: now also U7.13 (CSN_CFG3)
- net RUN_SAFE: now reaches R55.1
- net RUN_SAFE: now also U11.4 (Y)
- net RUN_BASE: now reaches R55.2, R56.1
- net RUN_BASE: now also Q14.1 (B)
- net BOOT_A2: now reaches C33.1
- net BOOT_A2: now also U7.35 (CA2)
- net MOTOR_A2: now reaches C33.2
- net MOTOR_A2: now also U7.37 (BMA2)
- net TMC_12V: now reaches C25.1
- net TMC_12V: now also U7.3 (12VOUT)
- net HW_ENABLE_24V: now reaches R57.1
- net DIR_IN: now reaches U9.1 (I1)
- net STOP_R: now reaches U9.3 (I0)
- net REFR_DIR: now reaches U9.4 (Y)
- net REFR_DIR: now also U7.18 (REFR_DIR)
- net SD_MODE: now reaches U9.6 (S)
- net SD_MODE: now also R36.1, U7.21 (SD_MODE), U8.6 (S)
- net DRV_EN_N: now reaches Q14.3 (C)
- net DRV_EN_N: now also R37.2, U7.28 (DRV_ENN)
- net TMC_5V: now reaches C26.1, U7.5 (5VOUT)
- net TMC_5V: now also R34.1
- net BOOT_A1: now reaches C32.1
- net BOOT_A1: now also U7.42 (CA1)
- net MOTOR_A1: now reaches C32.2
- net MOTOR_A1: now also U7.40 (BMA1)
- net VMOTOR_OK: now reaches U11.2 (B)
- net GH_B1_DRV: now reaches U7.1 (HB1)
- net SPI_SCK: now reaches U7.14 (SCK_CFG2)
- net SPI_MOSI: now reaches U7.15 (SDI_CFG1)
- net SPI_MISO: now reaches U7.16 (SDO_CFG0)
- net REFL_STEP: now reaches U7.17 (REFL_STEP)
- net REFL_STEP: now also U8.4 (Y)
- net ENC_B: now reaches U7.23 (ENCB_DCEN_CFG4)
- net ENC_A: now reaches U7.24 (ENCA_DCIN_CFG5)
- net ENC_I: now reaches U7.25 (ENCN_DCO_CFG6)
- net TMC_DIAG0: now reaches U7.26 (DIAG0_SWN)
- net TMC_DIAG1: now reaches U7.27 (DIAG1_SWP)
- net TMC_CPO: now reaches U7.31 (CPO)
- net TMC_CPO: now also C30.1
- net TMC_CPI: now reaches U7.32 (CPI)
- net TMC_CPI: now also C30.2
- net GH_A2_DRV: now reaches U7.36 (HA2)
- net GL_A2_DRV: now reaches U7.38 (LA2)
- net GL_A1_DRV: now reaches U7.39 (LA1)
- net GH_A1_DRV: now reaches U7.41 (HA1)
- net GH_B2_DRV: now reaches U7.44 (HB2)
- net GL_B2_DRV: now reaches U7.46 (LB2)
- net GL_B1_DRV: now reaches U7.47 (LB1)
- net SENSE_A: now reaches U7.8 (SRAH)
- net SENSE_B: now reaches U7.9 (SRBH)
- net STEP_IN: now reaches U8.1 (I1)
- net STOP_L: now reaches U8.3 (I0)

Commit message: Implement dual USB power/data ECO and consolidate industrial I/O
Parts:
- removed Q14: Q14, MMBT5551LT1G, symbol Custom:MMBT5551LT1G_NPN
- removed Q15: Q15, MMBT5551LT1G, symbol Custom:MMBT5551LT1G_NPN
- added Q14: Q14, MMBT5551LT1G, symbol Custom:MMBT5551LT1G
- added Q15: Q15, MMBT5551LT1G, symbol Custom:MMBT5551LT1G
Connections:
- net ENC_A is gone; now on net GND: U7.24 (ENCA_DCIN_CFG5)
- net ENC_B is gone; now on net GND: U7.23 (ENCB_DCEN_CFG4)
- net DRV_EN_N: now also Q14.3 (C)
- net ENABLE_CHAIN: now also Q14.2 (E), Q15.3 (C)
- net GND: now also Q15.2 (E)
- net HW_ENABLE_BASE: now also Q15.1 (B)
- net RUN_BASE: now also Q14.1 (B)
- net ENC_I: no longer names the net of U7.25 (ENCN_DCO_CFG6)
- no-connect marks 0 -> 1
Other:
- note removed: "ENC_A"
- note removed: "ENC_B"
- note removed: "ENC_I"

Commit message: Complete top-side routing and verify reference-board ECO
Connections:
- net RUN_SAFE: no longer U11.4 (Y)
- new net RUN_WINDOW_OK: U11.4 (Y)
Other:
- note added: "RUN_WINDOW_OK"
