File: dist/manufacturing/kicad-project/motion.kicad_sch (KiCad schematic)
At the start: 33 parts, among them Q14 Q14, Q15 Q15, U10 SN74LVC1G08DBVR, U11 SN74LVC1G08DBVR, U7 TMC5160A-TA-T, U8 74LVC1G157GW,125, U9 74LVC1G157GW,125

Commit message: Correct driver supply and brake protection power limits
Add the regulated 12 V TMC5160 gate supply and precision brake/OVP thresholds. Refresh top-side routing and manufacturing outputs with zero native DRC/ERC and complete connectivity. Verify native bypass paths and document calculations, sourcing, order holds, and unperformed powered tests.
Parts:
- C32, C33, C34, C35: value 220nF -> 470nF
Connections:
- net TMC_12V: now also C61.1, U7.4 (VSA)
- net VMOTOR: no longer C61.1, U7.4 (VSA)

Commit message: Fix source warnings and organize schematic on A4 sheets
Parts:
- removed C36, C37, C38, C39: 100nF, capacitor_cap0603, symbol Device:capacitor_down
- removed D1: D, BAV21W-7-F, symbol Device:diode_up
- removed Q14: Q14, MMBT5551LT1G, symbol Custom:MMBT5551LT1G
- removed Q15: Q15, MMBT5551LT1G, symbol Custom:MMBT5551LT1G
- removed R54, R56, R58: 10kΩ, resistor_res0603, symbol Device:boxresistor_down
- removed R55: 1kΩ, resistor_res0603, symbol Device:boxresistor_right
- removed R57: 100kΩ, resistor_res0603, symbol Device:boxresistor_right
- removed U10, U11: SN74LVC1G08DBVR, SN74LVC1G08DBVR, symbol Device:U_SN74LVC1G08DBVR
- removed U8, U9: 74LVC1G157GW,125, 74LVC1G157GW_125, symbol Device:U_74LVC1G157GW_125
Other:
- note added: "07 / Motion Controller"
- note added: "Bootstrap, charge-pump and local bypass parts are shown with the controller."
- note added: "U7 TMC5160A drives the external bridges; nominal regulated driver supply is 12 V."
- note removed: "04 / Motion Controller and Enable Chain"
- note removed: "DIR_IN"
- note removed: "ENABLE_CHAIN"
- note removed: "HW_ENABLE_24V"
- note removed: "HW_ENABLE_BASE"
- note removed: "MCU_RUN"
- note removed: "MOTOR_PG"
- note removed: "RUN_BASE"
- note removed: "RUN_PG"
- note removed: "RUN_SAFE"
- note removed: "RUN_WINDOW_OK"
- note removed: "SPI-controlled TMC5160A. Driver remains disabled until the hardware enable chain is valid."
- note removed: "STEP_IN"
- note removed: "STOP_L"
- note removed: "STOP_R"
- note removed: "U7: motion controller and gate driver. U8/U9: Step/Dir limit multiplexers. U10/U11 + Q14/Q15: hardwired enable interlock."
- note removed: "VMOTOR_OK"
