File: dist/manufacturing/kicad-project/motor_power.kicad_sch (KiCad schematic)
At the start: 52 parts, among them Q4 CSD19534Q5A, Q5 BSS123LT1G, U6 TPS26631RGER

Commit message: Complete orderable PD1180-EPR board release
Parts:
- removed C22, C23: 470uF, symbol Device:capacitor_polarized_right
- removed EFUSE_IN (x4): EFUSE_IN, symbol Custom:rail_up
- removed GND (x11): GND, symbol Custom:rail_down
- removed Q4: CSD19534Q5A, symbol Device:U_CSD19534Q5A
- removed Q5: BSS123LT1G, symbol Device:U_BSS123LT1G
- removed USB_VBUS (x4): USB_VBUS, symbol Custom:rail_up
- removed V3V3 (x2): V3V3, symbol Custom:rail_up
- removed VMON_ADC: VMON_ADC, symbol Custom:rail_up
- removed VMOTOR (x5): VMOTOR, symbol Custom:rail_up
- added C22, C23: 470uF, symbol Device:capacitor_polarized_down
- added EFUSE_IN (x3): EFUSE_IN, symbol Custom:rail_up
- added GND (x12): GND, symbol Custom:rail_down
- added Q4: Q4, symbol Custom:CSD19534Q5A_POWER_NMOS
- added Q5: Q5, symbol Custom:BSS123LT1G_NMOS
- added USB_VBUS (x4): USB_VBUS, symbol Custom:rail_up
- added V3V3 (x2): V3V3, symbol Custom:rail_up
- added VMOTOR (x5): VMOTOR, symbol Custom:rail_up
Connections:
- net IIN_MON: now also R26.1; no longer C19.1
- net at R28.2: now also C20.2, GND.1; no longer R24.2
- net at R33.2: now also GND.1
- net at C20.1: now also EFUSE_IN.1
- net at U6.1 (IN2), U6.2 (IN1): now also EFUSE_IN.1
- net at U6.17 (OUT2), U6.18 (OUT1): now also VMOTOR.1
- net at C18.2, U6.25 (EP): now also GND.1
- net at U6.5 (IN_SYS): now also USB_VBUS.1
- net at R22.1: now also USB_VBUS.1; no longer R19.1
- net at C19.2: now also GND.1
- net at C21.1: now also VMOTOR.1; no longer R31.1
- net at R21.2: now also GND.1
- net at R25.2: now also GND.1
- net at C24.2: now also GND.1
- net at R30.1: now also V3V3.1
- net at R26.2: now also GND.1
- net at R29.1: now also V3V3.1
- net at R27.1: now also VMOTOR.1
- net GND: no longer names the net of C21.2, U6.8 (GND)
- net GND: now also GND.1
- net OVP_TOP: no longer names the net of R22.2
- net VMON_MID: no longer names the net of R31.2
- new net: C22.1, VMOTOR.1
- new net: C22.2, GND.1
- new net: GND.1, R24.2
- new net: Q4.1 (source), Q4.2 (S2), Q4.3 (S3), USB_VBUS.1
- new net: Q4.4 (gate), Q5.3 (drain)
- new net: EFUSE_IN.1, Q4.5 (drain), Q4.6 (D2), Q4.7 (D3), Q4.8 (D4), Q4.9 (D5)
- new net: C23.1, VMOTOR.1
- new net: C23.2, GND.1
Other:
- note added: "Q4: reverse-blocking power MOSFET. Q5: fast gate clamp. U6: TPS26631 48 V eFuse, current monitor and fault output."

Commit message: Fix schematic style and top-side reset switch
Parts:
- removed EFUSE_IN (x3): EFUSE_IN, symbol Custom:rail_up
- removed GND (x12): GND, symbol Custom:rail_down
- removed USB_VBUS (x4): USB_VBUS, symbol Custom:rail_up
- removed V3V3 (x2): V3V3, symbol Custom:rail_up
- removed VMOTOR (x5): VMOTOR, symbol Custom:rail_up
- added EFUSE_IN (x3): EFUSE_IN, symbol Custom:rail_up
- added GND (x12): GND, symbol Custom:rail_down
- added USB_VBUS (x4): USB_VBUS, symbol Custom:rail_up
- added V3V3 (x2): V3V3, symbol Custom:rail_up
- added VMOTOR (x5): VMOTOR, symbol Custom:rail_up
Connections:
- net at R29.1: now also V3V3.1
- net at C20.1: now also EFUSE_IN.1
- net at C20.2, R28.2: now also GND.1
- net at C21.2, U6.8 (GND): now also GND.1
- net at R22.1: now also R19.1, USB_VBUS.1
- net at R25.2: now also GND.1
- net at C22.1: now also VMOTOR.1
- net at C22.2: now also GND.1
- net at R24.2: now also GND.1
- net at C21.1: now also R31.1, VMOTOR.1
- net at Q4.1 (S1), Q4.2 (S2), Q4.3 (S3): now also USB_VBUS.1
- net at Q4.5 (D1), Q4.6 (D2), Q4.7 (D3)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: now also EFUSE_IN.1
- net at U6.1 (IN2), U6.2 (IN1): now also EFUSE_IN.1
- net at U6.17 (OUT2), U6.18 (OUT1): now also VMOTOR.1
- net at C23.1: now also VMOTOR.1
- net at C23.2: now also GND.1
- net at Q5.2 (S): now also USB_VBUS.1
- net at R27.1: now also VMOTOR.1
- net at R30.1: now also V3V3.1
- net at U6.5 (IN_SYS): now also USB_VBUS.1
- net at C19.2: now also GND.1
- net at C18.2, U6.25 (EP): now also GND.1
- net at R33.2: now also GND.1
- net at R21.2: now also GND.1
- net at R26.2: now also GND.1
- net at C24.2: now also GND.1

Commit message: Use one USB-C port for PD and data
Parts:
- removed EFUSE_IN (x3): EFUSE_IN, symbol Custom:rail_up
- removed GND (x12): GND, symbol Custom:rail_down
- removed USB_VBUS (x4): USB_VBUS, symbol Custom:rail_up
- removed V3V3 (x2): V3V3, symbol Custom:rail_up
- removed VMOTOR (x5): VMOTOR, symbol Custom:rail_up
- added EFUSE_IN (x3): EFUSE_IN, symbol Custom:rail_up
- added GND (x12): GND, symbol Custom:rail_down
- added USB_VBUS (x4): USB_VBUS, symbol Custom:rail_up
- added V3V3 (x2): V3V3, symbol Custom:rail_up
- added VMOTOR (x5): VMOTOR, symbol Custom:rail_up
Connections:
- net at Q4.5 (D1), Q4.6 (D2), Q4.7 (D3)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: now also EFUSE_IN.1
- net at C22.1: now also VMOTOR.1
- net at R21.2: now also GND.1
- net at C20.2, R28.2: now also GND.1
- net at Q4.1 (S1), Q4.2 (S2), Q4.3 (S3): now also USB_VBUS.1
- net at C20.1: now also EFUSE_IN.1
- net at C21.1, R31.1: now also VMOTOR.1
- net at R29.1: now also V3V3.1
- net at U6.1 (IN2), U6.2 (IN1): now also EFUSE_IN.1
- net at C24.2: now also GND.1
- net at R19.1, R22.1: now also USB_VBUS.1
- net at R24.2: now also GND.1
- net at C18.2, U6.25 (EP): now also GND.1
- net at C23.1: now also VMOTOR.1
- net at R25.2: now also GND.1
- net at R26.2: now also GND.1
- net at C22.2: now also GND.1
- net at R27.1: now also VMOTOR.1
- net at C23.2: now also GND.1
- net at Q5.2 (S): now also USB_VBUS.1
- net at U6.17 (OUT2), U6.18 (OUT1): now also VMOTOR.1
- net at C21.2, U6.8 (GND): now also GND.1
- net at R30.1: now also V3V3.1
- net at C19.2: now also GND.1
- net at R33.2: now also GND.1
- net at U6.5 (IN_SYS): now also USB_VBUS.1

Commit message: fix: finalize single-port EPR controller
Parts:
- removed EFUSE_IN (x3): EFUSE_IN, symbol Custom:rail_up
- removed GND (x12): GND, symbol Custom:rail_down
- removed USB_VBUS (x4): USB_VBUS, symbol Custom:rail_up
- removed V3V3 (x2): V3V3, symbol Custom:rail_up
- removed VMOTOR (x5): VMOTOR, symbol Custom:rail_up
- C18, C19, C20, C24: footprint (none) -> capacitor_cap0603
- C21: footprint (none) -> capacitor_cap1206
- C22, C23: footprint (none) -> EEUFR1J471
- Q4: footprint (none) -> CSD19534Q5A
- Q5: footprint (none) -> BSS123LT1G
- R19, R20, R21, R22, R23, R24, R25, R26, R27, R28, R29, R30, R31, R32, R33: footprint (none) -> resistor_res0603
- U6: footprint (none) -> TPS26631RGER
Connections:
- net EFUSE_FAULT_N: now also U6.14 (N_FLT)
- net IIN_MON: now also C19.1, U6.13 (IMON)
- net ILIM_SET: now also U6.10 (ILIM)
- net GND: now reaches C23.2
- net GND: now also C18.2, C19.2, C20.2, C21.2, C22.2, C24.2, R21.2, R24.2, R25.2, R26.2, R28.2, R33.2, U6.25 (EP), U6.8 (GND)
- net VMOTOR: now reaches C22.1
- net VMOTOR: now also C21.1, C23.1, R27.1, R31.1, U6.17 (OUT2), U6.18 (OUT1)
- net PG_DIV: now reaches R27.2, U6.15 (PGTH)
- net PG_DIV: now also R28.1
- net USB_VBUS: now reaches Q4.1 (S1), Q4.2 (S2), Q4.3 (S3)
- net USB_VBUS: now also Q5.2 (S), R19.1, R22.1, U6.5 (IN_SYS)
- net VMON_MID: now reaches R32.1
- net VMON_MID: now also R31.2
- net VMON_ADC: now reaches R32.2
- net VMON_ADC: now also C24.1, R33.1
- net V3V3: now reaches R30.1
- net V3V3: now also R29.1
- net UVLO_MID: now reaches R20.1
- net UVLO_MID: now also R19.2
- net UVLO_DIV: now reaches R20.2, R21.1
- net UVLO_DIV: now also U6.6 (UVLO)
- net EFUSE_IN: now reaches U6.1 (IN2), U6.2 (IN1)
- net EFUSE_IN: now also C20.1, Q4.5 (D1), Q4.6 (D2), Q4.7 (D3), Q4.8 (D4), Q4.9 (D5)
- net EFUSE_EN: now reaches U6.12 (N_SHDN)
- net MOTOR_PG: now reaches U6.16 (PGOOD)
- net MOTOR_PG: now also R29.2
- net BLOCK_GATE: now reaches U6.3 (B_GATE)
- net BLOCK_GATE: now also Q4.4 (G), Q5.3 (D)
- net BLOCK_FAST_GATE: now reaches U6.4 (DRV)
- net BLOCK_FAST_GATE: now also Q5.1 (G)
- net OVP_DIV: now reaches U6.7 (OVP)
- net OVP_DIV: now also R23.2, R24.1
- net SLEW_CAP: now reaches U6.9 (dVdT)
- net SLEW_CAP: now also C18.1
- net OVP_TOP: now reaches R22.2
- net OVP_TOP: now also R23.1
- no-connect marks 0 -> 7

Commit message: Implement dual USB power/data ECO and consolidate industrial I/O
Parts:
- removed Q4: Q4, CSD19534Q5A, symbol Custom:CSD19534Q5A_POWER_NMOS
- removed Q5: Q5, BSS123LT1G, symbol Custom:BSS123LT1G_NMOS
- added Q4: CSD19534Q5A, CSD19534Q5A, symbol Device:U_CSD19534Q5A
- added Q5: Q5, BSS123LT1G, symbol Custom:BSS123LT1G
Connections:
- net BLOCK_FAST_GATE: now also Q5.1 (G)
- net BLOCK_GATE: now also Q4.4 (G), Q5.3 (D)
- net EFUSE_IN: now also Q4.5 (D1), Q4.6 (D2), Q4.7 (D3), Q4.8 (D4), Q4.9 (D5)
- net USB_VBUS renamed PD_VBUS
- net PD_VBUS: now also Q4.1 (S1), Q4.2 (S2), Q4.3 (S3), Q5.2 (S)
