File: dist/manufacturing/kicad-project/outputs.kicad_sch (KiCad schematic)
At the start: 15 parts, among them J9 B4B-PH-K-S(LF)(SN), Q24 MMBT5551LT1G, Q25 MMBT5551LT1G

Commit message: Complete orderable PD1180-EPR board release
Parts:
- removed GND (x3): GND, symbol Custom:rail_down
- removed Q24, Q25: MMBT5551LT1G, symbol Device:U_MMBT5551LT1G
- removed VMOTOR (x3): VMOTOR, symbol Custom:rail_up
- added GND (x2): GND, symbol Custom:rail_down
- added Q24: Q24, symbol Custom:MMBT5551LT1G_NPN
- added Q25: Q25, symbol Custom:MMBT5551LT1G_NPN
- added VMOTOR (x3): VMOTOR, symbol Custom:rail_up
Connections:
- net at D12.1 (2): now also VMOTOR.1
- net at R99.1: now also Q24.1 (base)
- net at R99.2: now also GND.1, Q24.2 (emitter)
- net at D11.1 (2): now also VMOTOR.1
- net at D12.2 (1): now also Q25.3 (collector)
- net at R100.2: no longer R101.1
- net at R101.2: now also GND.1, Q25.2 (emitter)
- net at J9.1: now also VMOTOR.1
- net at D11.2 (1): now also Q24.3 (collector)
- new net: Q25.1 (base), R101.1
Other:
- note added: "Q24/Q25: open-collector 24 V output drivers; base pulldowns keep outputs off during reset."

Commit message: Fix schematic style and top-side reset switch
Parts:
- removed GND (x2): GND, symbol Custom:rail_down
- removed VMOTOR (x3): VMOTOR, symbol Custom:rail_up
- added GND (x2): GND, symbol Custom:rail_down
- added VMOTOR (x3): VMOTOR, symbol Custom:rail_up
Connections:
- net at J9.1: now also VMOTOR.1
- net at D11.1 (2): now also VMOTOR.1
- net at Q24.2 (E), R99.2: now also GND.1
- net at Q25.2 (E), R101.2: now also GND.1
- net at D12.1 (2): now also VMOTOR.1

Commit message: Use one USB-C port for PD and data
Parts:
- removed GND (x2): GND, symbol Custom:rail_down
- removed VMOTOR (x3): VMOTOR, symbol Custom:rail_up
- added GND (x2): GND, symbol Custom:rail_down
- added VMOTOR (x3): VMOTOR, symbol Custom:rail_up
Connections:
- net at J9.1: now also VMOTOR.1
- net at D11.1 (2): now also VMOTOR.1
- net at Q24.2 (E), R99.2: now also GND.1
- net at D12.1 (2): now also VMOTOR.1
- net at Q25.2 (E), R101.2: now also GND.1
Changed lines of the file:
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@@
     (instances
       (project ""
-        (path "/17a83a49-7a29-40ba-a4d1-006f579ceb16/23dc544b-a034-4538-975a-7104760a6a9a"
+        (path "/3270f766-a91f-4ae6-bf4b-7f3cb477ac52/4cfb473c-a801-482f-8c22-a948a8246465"
           (reference "J9")
           (unit 1)
@@
     (instances
       (project ""
-        (path "/17a83a49-7a29-40ba-a4d1-006f579ceb16/23dc544b-a034-4538-975a-7104760a6a9a"
+        (path "/3270f766-a91f-4ae6-bf4b-7f3cb477ac52/4cfb473c-a801-482f-8c22-a948a8246465"
           (reference "Q24")
           (unit 1)
@@
     (instances
       (project ""
-        (path "/17a83a49-7a29-40ba-a4d1-006f579ceb16/23dc544b-a034-4538-975a-7104760a6a9a"
+        (path "/3270f766-a91f-4ae6-bf4b-7f3cb477ac52/4cfb473c-a801-482f-8c22-a948a8246465"
           (reference "R98")
           (unit 1)
@@
     (instances
       (project ""
-        (path "/17a83a49-7a29-40ba-a4d1-006f579ceb16/23dc544b-a034-4538-975a-7104760a6a9a"
+        (path "/3270f766-a91f-4ae6-bf4b-7f3cb477ac52/4cfb473c-a801-482f-8c22-a948a8246465"
           (reference "R99")
           (unit 1)
@@
     (instances
       (project ""
-        (path "/17a83a49-7a29-40ba-a4d1-006f579ceb16/23dc544b-a034-4538-975a-7104760a6a9a"
+        (path "/3270f766-a91f-4ae6-bf4b-7f3cb477ac52/4cfb473c-a801-482f-8c22-a948a8246465"
           (reference "D11")
           (unit 1)
@@
     (instances
       (project ""
-        (path "/17a83a49-7a29-40ba-a4d1-006f579ceb16/23dc544b-a034-4538-975a-7104760a6a9a"
+        (path "/3270f766-a91f-4ae6-bf4b-7f3cb477ac52/4cfb473c-a801-482f-8c22-a948a8246465"
           (reference "Q25")
           (unit 1)
@@
     (instances
       (project ""
-        (path "/17a83a49-7a29-40ba-a4d1-006f579ceb16/23dc544b-a034-4538-975a-7104760a6a9a"
+        (path "/3270f766-a91f-4ae6-bf4b-7f3cb477ac52/4cfb473c-a801-482f-8c22-a948a8246465"
           (reference "R100")
           (unit 1)
@@
     (instances
       (project ""
-        (path "/17a83a49-7a29-40ba-a4d1-006f579ceb16/23dc544b-a034-4538-975a-7104760a6a9a"
+        (path "/3270f766-a91f-4ae6-bf4b-7f3cb477ac52/4cfb473c-a801-482f-8c22-a948a8246465"
           (reference "R101")
           (unit 1)
@@
     (instances
       (project ""
-        (path "/17a83a49-7a29-40ba-a4d1-006f579ceb16/23dc544b-a034-4538-975a-7104760a6a9a"
+        (path "/3270f766-a91f-4ae6-bf4b-7f3cb477ac52/4cfb473c-a801-482f-8c22-a948a8246465"
           (reference "D12")
           (unit 1)
@@
     (instances
       (project ""
-        (path "/17a83a49-7a29-40ba-a4d1-006f579ceb16/23dc544b-a034-4538-975a-7104760a6a9a"
+        (path "/3270f766-a91f-4ae6-bf4b-7f3cb477ac52/4cfb473c-a801-482f-8c22-a948a8246465"
           (reference "VMOTOR")
           (unit 1)
@@
     (instances
       (project ""
-        (path "/17a83a49-7a29-40ba-a4d1-006f579ceb16/23dc544b-a034-4538-975a-7104760a6a9a"
+        (path "/3270f766-a91f-4ae6-bf4b-7f3cb477ac52/4cfb473c-a801-482f-8c22-a948a8246465"
           (reference "VMOTOR")
           (unit 1)
@@
     (instances
       (project ""
-        (path "/17a83a49-7a29-40ba-a4d1-006f579ceb16/23dc544b-a034-4538-975a-7104760a6a9a"
+        (path "/3270f766-a91f-4ae6-bf4b-7f3cb477ac52/4cfb473c-a801-482f-8c22-a948a8246465"
           (reference "VMOTOR")
           (unit 1)
@@
     (instances
       (project ""
-        (path "/17a83a49-7a29-40ba-a4d1-006f579ceb16/23dc544b-a034-4538-975a-7104760a6a9a"
+        (path "/3270f766-a91f-4ae6-bf4b-7f3cb477ac52/4cfb473c-a801-482f-8c22-a948a8246465"
           (reference "GND")
           (unit 1)
@@
     (instances
       (project ""
-        (path "/17a83a49-7a29-40ba-a4d1-006f579ceb16/23dc544b-a034-4538-975a-7104760a6a9a"
+        (path "/3270f766-a91f-4ae6-bf4b-7f3cb477ac52/4cfb473c-a801-482f-8c22-a948a8246465"
           (reference "GND")
           (unit 1)

Commit message: fix: finalize single-port EPR controller
Parts:
- removed GND (x2): GND, symbol Custom:rail_down
- removed VMOTOR (x3): VMOTOR, symbol Custom:rail_up
- D11, D12: value SS110 -> D; footprint (none) -> SS110
- J9: value B4B-PH-K-S(LF)(SN) -> J9; footprint (none) -> B4B-PH-K-S_LF_SN
- Q24, Q25: footprint (none) -> MMBT5551LT1G
- R100, R101, R98, R99: footprint (none) -> resistor_res0603
Connections:
- net GND: now reaches Q24.2 (E), R99.2
- net GND: now also Q25.2 (E), R101.2
- net VMOTOR: now reaches D11.1 (2)
- net VMOTOR: now also D12.1 (2), J9.1
- net OUT0: now reaches D11.2 (1), Q24.3 (C)
- net OUT0: now also J9.3
- net HW_ENABLE_24V: now reaches J9.2
- net OUT1: now reaches J9.4
- net OUT1: now also D12.2 (1), Q25.3 (C)
- net OUT0_BASE: now reaches Q24.1 (B), R99.1
- net OUT0_BASE: now also R98.2
- net OUT1_BASE: now reaches Q25.1 (B), R101.1
- net OUT1_BASE: now also R100.2
- net OUT0_DRIVE: now reaches R98.1
- net OUT1_DRIVE: now reaches R100.1

Commit message: Implement dual USB power/data ECO and consolidate industrial I/O
Parts:
- removed J9: J9, B4B-PH-K-S_LF_SN, symbol Device:J_B4B-PH-K-S_LF_SN
- removed Q24: Q24, MMBT5551LT1G, symbol Custom:MMBT5551LT1G_NPN
- removed Q25: Q25, MMBT5551LT1G, symbol Custom:MMBT5551LT1G_NPN
- added Q24: Q24, MMBT5551LT1G, symbol Custom:MMBT5551LT1G
- added Q25: Q25, MMBT5551LT1G, symbol Custom:MMBT5551LT1G
Connections:
- net GND: now also Q24.2 (E), Q25.2 (E)
- net OUT0: now also Q24.3 (C)
- net OUT0_BASE: now also Q24.1 (B)
- net OUT1: now also Q25.3 (C)
- net OUT1_BASE: now also Q25.1 (B)
Other:
- note added: "13 / Hardware Enable and Outputs"
- note added: "J7: motor rail, 24 V hardware enable, OUT0 and OUT1. External loads need rating review."
- note removed: "12 / Hardware Enable and Outputs"
- note removed: "HW_ENABLE_24V"
- note removed: "J9: motor rail, 24 V hardware enable, OUT0 and OUT1. External loads need rating review."
