File: dist/manufacturing/kicad-project/outputs.kicad_sch (KiCad schematic)
At the start: 8 parts, among them Q24 Q24, Q25 Q25

Commit message: Fix source warnings and organize schematic on A4 sheets
Parts:
- Q24: value Q24 -> MMBT5551LT1G
- Q25: value Q25 -> MMBT5551LT1G
Other:
- note added: "20 / Hardware Outputs"
- note added: "J7 carries OUT0/OUT1. External load and duty ratings still require system qualification."
- note added: "Q24/Q25 provide the two open-collector outputs; base pulldowns keep reset inactive."
- note removed: "13 / Hardware Enable and Outputs"
- note removed: "J7: motor rail, 24 V hardware enable, OUT0 and OUT1. External loads need rating review."
- note removed: "Q24/Q25: open-collector 24 V output drivers; base pulldowns keep outputs off during reset."
Changed lines of the file:
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@@
       )
     )
-    (property "Value" "Q24"
+    (property "Value" "MMBT5551LT1G"
       (id 1)
       (at 175.08749999999998 230.175 0)
@@
     (instances
       (project ""
-        (path "/888afcaf-aca0-4ec5-ab90-6fb77de6f3f5/bf747cd2-f085-4953-aa3c-cf8d4192d869"
+        (path "/9ce6d0ce-044d-4e77-ac59-1290d960b5b5/957b127e-e625-4eb1-986b-191490207d6c"
           (reference "Q24")
           (unit 1)
@@
     (instances
       (project ""
-        (path "/888afcaf-aca0-4ec5-ab90-6fb77de6f3f5/bf747cd2-f085-4953-aa3c-cf8d4192d869"
+        (path "/9ce6d0ce-044d-4e77-ac59-1290d960b5b5/957b127e-e625-4eb1-986b-191490207d6c"
           (reference "R98")
           (unit 1)
@@
     (instances
       (project ""
-        (path "/888afcaf-aca0-4ec5-ab90-6fb77de6f3f5/bf747cd2-f085-4953-aa3c-cf8d4192d869"
+        (path "/9ce6d0ce-044d-4e77-ac59-1290d960b5b5/957b127e-e625-4eb1-986b-191490207d6c"
           (reference "R99")
           (unit 1)
@@
     (instances
       (project ""
-        (path "/888afcaf-aca0-4ec5-ab90-6fb77de6f3f5/bf747cd2-f085-4953-aa3c-cf8d4192d869"
+        (path "/9ce6d0ce-044d-4e77-ac59-1290d960b5b5/957b127e-e625-4eb1-986b-191490207d6c"
           (reference "D11")
           (unit 1)
@@
     (property "Reference" "Q25"
       (id 0)
-      (at 430.08750000000003 205.125 0)
-      (effects
-        (font
-          (size 1.27 1.27)
-        )
-        (hide yes)
-      )
-    )
-    (property "Value" "Q25"
-      (id 1)
-      (at 430.08750000000003 230.175 0)
+      (at 430.0875 205.125 0)
+      (effects
+        (font
+          (size 1.27 1.27)
+        )
+        (hide yes)
+      )
+    )
+    (property "Value" "MMBT5551LT1G"
+      (id 1)
+      (at 430.0875 230.175 0)
       (effects
         (font
@@
     (property "Footprint" "MMBT5551LT1G"
       (id 2)
-      (at 428.3095 217.65 90)
-      (effects
-        (font
-          (size 1.27 1.27)
-        )
-        (hide yes)
-      )
-    )
-    (property "Datasheet" "~"
-      (id 3)
-      (at 430.08750000000003 217.65 0)
-      (effects
-        (font
-          (size 1.27 1.27)
-        )
-        (hide yes)
-      )
-    )
-    (property "Description" ""
-      (id 4)
-      (at 430.08750000000003 217.65 0)
+      (at 428.30949999999996 217.65 90)
+      (effects
+        (font
+          (size 1.27 1.27)
+        )
+        (hide yes)
+      )
+    )
+    (property "Datasheet" "~"
+      (id 3)
+      (at 430.0875 217.65 0)
+      (effects
+        (font
+          (size 1.27 1.27)
+        )
+        (hide yes)
+      )
+    )
+    (property "Description" ""
+      (id 4)
+      (at 430.0875 217.65 0)
       (effects
         (font
@@
     (instances
       (project ""
-        (path "/888afcaf-aca0-4ec5-ab90-6fb77de6f3f5/bf747cd2-f085-4953-aa3c-cf8d4192d869"
+        (path "/9ce6d0ce-044d-4e77-ac59-1290d960b5b5/957b127e-e625-4eb1-986b-191490207d6c"
           (reference "Q25")
           (unit 1)
@@
     (instances
       (project ""
-        (path "/888afcaf-aca0-4ec5-ab90-6fb77de6f3f5/bf747cd2-f085-4953-aa3c-cf8d4192d869"
+        (path "/9ce6d0ce-044d-4e77-ac59-1290d960b5b5/957b127e-e625-4eb1-986b-191490207d6c"
           (reference "R100")
           (unit 1)
@@
     (instances
       (project ""
-        (path "/888afcaf-aca0-4ec5-ab90-6fb77de6f3f5/bf747cd2-f085-4953-aa3c-cf8d4192d869"
+        (path "/9ce6d0ce-044d-4e77-ac59-1290d960b5b5/957b127e-e625-4eb1-986b-191490207d6c"
           (reference "R101")
           (unit 1)
@@
     (property "Value" "D"
       (id 1)
-      (at 489.97499999999997 172.65 0)
+      (at 489.975 172.65 0)
       (effects
         (font
@@
     (instances
       (project ""
-        (path "/888afcaf-aca0-4ec5-ab90-6fb77de6f3f5/bf747cd2-f085-4953-aa3c-cf8d4192d869"
+        (path "/9ce6d0ce-044d-4e77-ac59-1290d960b5b5/957b127e-e625-4eb1-986b-191490207d6c"
           (reference "D12")
           (unit 1)
@@
     )
   )
-  (text "13 / Hardware Enable and Outputs"
-    (at 113.625 97.65 0)
-    (effects
-      (font
-        (size 1.27 1.27)
-        (color 0 0 0 1)
-      )
-    )
-  )
-  (text "J7: motor rail, 24 V hardware enable, OUT0 and OUT1. External loads need rating review."
-    (at 113.625 118.65 0)
-    (effects
-      (font
-        (size 1.27 1.27)
-        (color 0 0 0 1)
-      )
-    )
-  )
-  (text "Q24/Q25: open-collector 24 V output drivers; base pulldowns keep outputs off during reset."
-    (at 113.625 130.65 0)
+  (text "20 / Hardware Outputs"
+    (at 308.625 49.650000000000006 0)
+    (effects
+      (font
+        (size 1.27 1.27)
+        (color 0 0 0 1)
+      )
+    )
+  )
+  (text "Q24/Q25 provide the two open-collector outputs; base pulldowns keep reset inactive."
+    (at 308.625 67.65 0)
+    (effects
+      (font
+        (size 1.27 1.27)
+        (color 0 0 0 1)
+      )
+    )
+  )
+  (text "J7 carries OUT0/OUT1. External load and duty ratings still require system qualification."
+    (at 308.625 78.15 0)
     (effects
       (font
@@
   )
   (text "OUT0"
-    (at 229.42499999999998 181.95000000000002 -90)
+    (at 229.425 181.95000000000002 -90)
     (effects
       (font
@@
   )
   (text "OUT0_BASE"
-    (at 146.92499999999998 230.4 -90)
+    (at 146.92499999999998 230.40000000000003 -90)
     (effects
       (font
@@
   )
   (text "OUT1_BASE"
-    (at 401.92499999999995 230.4 -90)
+    (at 401.925 230.40000000000003 -90)
     (effects
       (font
@@
   )
   (text "OUT1"
-    (at 433.95000000000005 197.1 -90)
+    (at 433.95 197.1 -90)
     (effects
       (font
@@
   )
   (text "OUT1"
-    (at 484.425 181.95000000000002 -90)
-    (effects
-      (font
+    (at 484.42499999999995 181.95000000000002 -90)
+    (effects
+      (font
