File: dist/manufacturing/kicad-project/bridge_a.kicad_sch (KiCad schematic)
At the start: 14 parts, among them J2 J2, Q6 CSD19534Q5A, Q7 CSD19534Q5A, Q8 CSD19534Q5A, Q9 CSD19534Q5A

Commit message: Fix source warnings and organize schematic on A4 sheets
Parts:
- removed Q6, Q7, Q8, Q9: CSD19534Q5A, CSD19534Q5A, symbol Device:U_CSD19534Q5A
- added Q6, Q7, Q8, Q9: CSD19534Q5A, CSD19534Q5A, symbol Custom:CSD19534Q5A
- J2: value J2 -> B4P-VH(LF)(SN)
Connections:
- net GH_A1: now also Q6.4 (G)
- net GH_A2: now also Q8.4 (G)
- net GL_A1: now also Q7.4 (G)
- net GL_A2: now also Q9.4 (G)
- net MOTOR_A1: now also Q6.1 (S1), Q6.2 (S2), Q6.3 (S3), Q7.5 (D1), Q7.6 (D2), Q7.7 (D3), Q7.8 (D4), Q7.9 (D5)
- net MOTOR_A2: now also Q8.1 (S1), Q8.2 (S2), Q8.3 (S3), Q9.5 (D1), Q9.6 (D2), Q9.7 (D3), Q9.8 (D4), Q9.9 (D5)
- net SENSE_A: now also Q7.1 (S1), Q7.2 (S2), Q7.3 (S3), Q9.1 (S1), Q9.2 (S2), Q9.3 (S3)
- net VMOTOR: now also Q6.5 (D1), Q6.6 (D2), Q6.7 (D3), Q6.8 (D4), Q6.9 (D5), Q8.5 (D1), Q8.6 (D2), Q8.7 (D3), Q8.8 (D4), Q8.9 (D5)
Other:
- note added: "09 / Motor Phase A Power Bridge"
- note added: "J2 connects both motor windings. The 5.5 A RMS design target is not a qualified setting."
- note added: "Q6/Q8 high-side and Q7/Q9 low-side switches form phase A; R109 is the Kelvin shunt."
- note removed: "05 / Motor Phase A Power Bridge"
- note removed: "Phase A target 5.5 A RMS; Kelvin sense routing and high-current copper require review."
- note removed: "Q6/Q8: high-side MOSFETs. Q7/Q9: low-side MOSFETs. R109: 33 mOhm, 3 W phase-current shunt."
