File: dist/manufacturing/kicad-project/bridge_b.kicad_sch (KiCad schematic)
At the start: 13 parts, among them Q10 CSD19534Q5A, Q11 CSD19534Q5A, Q12 CSD19534Q5A, Q13 CSD19534Q5A

Commit message: Fix source warnings and organize schematic on A4 sheets
Parts:
- removed Q10, Q11, Q12, Q13: CSD19534Q5A, CSD19534Q5A, symbol Device:U_CSD19534Q5A
- added Q10, Q11, Q12, Q13: CSD19534Q5A, CSD19534Q5A, symbol Custom:CSD19534Q5A
Connections:
- net GH_B1: now also Q10.4 (G)
- net GH_B2: now also Q12.4 (G)
- net GL_B1: now also Q11.4 (G)
- net GL_B2: now also Q13.4 (G)
- net MOTOR_B1: now also Q10.1 (S1), Q10.2 (S2), Q10.3 (S3), Q11.5 (D1), Q11.6 (D2), Q11.7 (D3), Q11.8 (D4), Q11.9 (D5)
- net MOTOR_B2: now also Q12.1 (S1), Q12.2 (S2), Q12.3 (S3), Q13.5 (D1), Q13.6 (D2), Q13.7 (D3), Q13.8 (D4), Q13.9 (D5)
- net SENSE_B: now also Q11.1 (S1), Q11.2 (S2), Q11.3 (S3), Q13.1 (S1), Q13.2 (S2), Q13.3 (S3)
- net VMOTOR: now also Q10.5 (D1), Q10.6 (D2), Q10.7 (D3), Q10.8 (D4), Q10.9 (D5), Q12.5 (D1), Q12.6 (D2), Q12.7 (D3), Q12.8 (D4), Q12.9 (D5)
Other:
- note added: "10 / Motor Phase B Power Bridge"
- note added: "Q10/Q12 high-side and Q11/Q13 low-side switches form phase B."
- note added: "R110 is the independent 33 mOhm shunt; preserve the Kelvin sense connections."
- note removed: "06 / Motor Phase B Power Bridge"
- note removed: "Phase B target 5.5 A RMS; independent 33 milliohm sense resistor."
- note removed: "Q10/Q12: high-side MOSFETs. Q11/Q13: low-side MOSFETs. R110: 33 mOhm, 3 W phase-current shunt."
