File: dist/manufacturing/kicad-project/logic_power.kicad_sch (KiCad schematic)
At the start: 30 parts, among them U22 LMR36510ADDAR, U23 LM66100DCKR, U24 LM66100DCKR, U5 LMR36510ADDAR

Commit message: Fix source warnings and organize schematic on A4 sheets
Parts:
- removed C62: 2.2uF, capacitor_cap1206, symbol Device:capacitor_down
- removed C63, C69, C70: 100nF, capacitor_cap0603, symbol Device:capacitor_down
- removed C64: 1uF, capacitor_cap0603, symbol Device:capacitor_down
- removed C65: 100nF, capacitor_cap0603, symbol Device:capacitor_right
- removed C66, C67, C68: 22uF, capacitor_cap0805, symbol Device:capacitor_down
- removed C71: 10uF, capacitor_cap0603, symbol Device:capacitor_down
- removed L2: 22µH, SWPA6045S220MT, symbol Device:inductor_right
- removed R102: 100kΩ, resistor_res0603, symbol Device:boxresistor_down
- removed R103: 43.2kΩ, resistor_res0603, symbol Device:boxresistor_down
- removed R104, R111: 10kΩ, resistor_res0603, symbol Device:boxresistor_down
- removed U22: LMR36510ADDAR, LMR36510ADDAR, symbol Device:U_LMR36510ADDAR
- removed U23, U24: LM66100DCKR, LM66100DCKR, symbol Device:U_LM66100DCKR
Connections:
- no-connect marks 2 -> 0
Other:
- note added: "03 / PD Backup Supply"
- note added: "Input spans default USB 5 V through the specified 48 V EPR operating target."
- note added: "U5 converts PD VBUS to V3V3_PD; L1 and its feedback/bypass network are shown here."
- note removed: "02 / PD and Motor Backup Supplies"
- note removed: "LOGIC_OR_PRIORITY"
- note removed: "MOTOR_BUCK_BOOT"
- note removed: "MOTOR_BUCK_FB"
- note removed: "MOTOR_BUCK_SW"
- note removed: "MOTOR_BUCK_VCC"
- note removed: "MOTOR_LOGIC_PG"
- note removed: "PD VBUS or DATA USB starts logic; the motor-bus buck retains brake-control backup after PD loss."
- note removed: "U5: PD 5-48 V buck. U22: VMOTOR backup buck. U23/U24 + R111: status-interlocked OR into board V3V3; U26/U27 power the separate MCU rail."
