File: dist/manufacturing/kicad-project/serial.kicad_sch (KiCad schematic)
At the start: 14 parts, among them U19 TCAN332DR, U20 MAX3485EESA+T, U21 MAX3232ESE+T

Commit message: Fix source warnings and organize schematic on A4 sheets
Parts:
- removed C56, C57: 100nF, capacitor_cap0603, symbol Device:capacitor_right
- removed C58, C59, C60: 100nF, capacitor_cap0603, symbol Device:capacitor_down
- removed U21: MAX3232ESE+T, MAX3232ESE_T, symbol Device:U_MAX3232ESE_T
Connections:
- no-connect marks 4 -> 2
Other:
- note added: "18 / CAN and RS485"
- note added: "J7 carries both buses; termination and RS485 bias are defined at the system level."
- note added: "U19 is the 3.3 V CAN transceiver; U20 is RS485. D2/D3 provide line protection."
- note removed: "12 / CAN, RS485 and RS232"
- note removed: "External CAN/RS485 termination; J7 carries RS232, CAN and RS485."
- note removed: "RS232_C1N"
- note removed: "RS232_C1P"
- note removed: "RS232_C2N"
- note removed: "RS232_C2P"
- note removed: "RS232_RX"
- note removed: "RS232_RX_CONN"
- note removed: "RS232_TX"
- note removed: "RS232_TX_CONN"
- note removed: "RS232_VN"
- note removed: "RS232_VP"
- note removed: "U19: 3.3 V CAN transceiver; D2: CAN TVS. U20: RS485 transceiver; D3: RS485 TVS. U21: RS232 transceiver."
