File: dist/manufacturing/kicad-project/telemetry.kicad_sch (KiCad schematic)
At the start: 17 parts, among them U29 TMP102AIDRLR, U30 ADS1115IDGSR, U31 INA240A1DR, U32 INA240A1DR, U33 SN74LVC1G08DBVR

Commit message: Fix source warnings and organize schematic on A4 sheets
Parts:
- removed C81, C82: 100nF, capacitor_cap0603, symbol Device:capacitor_down
- removed C83, C84: 10nF, capacitor_cap0603, symbol Device:capacitor_down
- removed R115, R116: 5mΩ, FRM121WFR005TM, symbol Device:boxresistor_right
- removed R117, R118: 1kΩ, resistor_res0603, symbol Device:boxresistor_right
- removed U31, U32: INA240A1DR, INA240A1DR, symbol Device:U_INA240A1DR
Connections:
- no-connect marks 3 -> 1
Other:
- note added: "22 / Temperature and Bus Diagnostics"
- note added: "Sensor addresses are 0x48 and 0x49. Temperature correlation requires load testing."
- note added: "U29 TMP102 senses temperature; U33 provides hardware inhibit. U30 ADS1115 monitors the bus."
- note removed: "15 / Temperature and Current Diagnostics"
- note removed: "MOTOR_A1"
- note removed: "MOTOR_A1_OUT"
- note removed: "MOTOR_B1"
- note removed: "MOTOR_B1_OUT"
- note removed: "PHASE_A_ADC"
- note removed: "PHASE_A_RAW"
- note removed: "PHASE_B_ADC"
- note removed: "PHASE_B_RAW"
- note removed: "U29: power-stage temperature, address 0x48. U33: temperature hardware inhibit. U30: bus-monitor ADC, address 0x49."
- note removed: "U31/U32: bidirectional winding telemetry, 20 V/V across 5 mOhm = 100 mV/A, centered at 1.65 V. Not a short-circuit trip."
