File: dist/manufacturing/kicad-project/usb_logic.kicad_sch (KiCad schematic)
At the start: 13 parts, among them U25 TLV75533PDBVR, U26 LM66100DCKR, U27 LM66100DCKR, U28 TPS2553DBVR

Commit message: Fix source warnings and organize schematic on A4 sheets
Other:
- note added: "21 / USB Logic Power"
- note added: "R119/R120 sense board supply on PB1. Industrial peripherals require board power."
- note added: "U28 limits DATA power; U25 regulates V3V3_USB. U26/U27 reverse-block the MCU rail."
- note removed: "14 / USB Logic Power"
- note removed: "U26/U27: reverse-blocked V3V3_MCU. R119/R120 sense board power on PB1; PD status is polled."
- note removed: "U28: DATA current limiter. U25: 3.3 V LDO. DATA powers MCU only; peripherals require board power."
