File: dist/manufacturing/kicad-project/indicators.kicad_sch (KiCad schematic)
At the start: 15 parts, among them Q26 AO3400A, U35 TCA9538PWR

Commit message: Fix source warnings and organize schematic on A4 sheets
Parts:
- removed BZ1: FUET-9650B-3V, FUET-9650B-3V, symbol Custom:FUET-9650B-3V
- removed C96: 10uF, capacitor_cap0603, symbol Device:capacitor_down
- removed D16: NH-B2020RGBA-HF, NH-B2020RGBA-HF, symbol Device:U_NH-B2020RGBA-HF
- removed D18: D, BAV21W-7-F, symbol Device:diode_up
- removed Q26: AO3400A, AO3400A, symbol Custom:AO3400A
- removed R126: 1kΩ, resistor_res0603, symbol Device:boxresistor_right
- removed R127: 100kΩ, resistor_res0603, symbol Device:boxresistor_down
- added D16: NH-B2020RGBA-HF, NH-B2020RGBA-HF, symbol Custom:NH-B2020RGBA-HF
Connections:
- net RGB_B_K: now also D16.2 (B_K)
- net RGB_G_K: now also D16.4 (G_K)
- net RGB_R_K: now also D16.1 (R_K)
- net V3V3: now also D16.3 (A)
Other:
- note added: "25 / Status and Independent Power Indication"
- note added: "D17 shows board V3V3 independently of firmware; USB-only MCU power is distinct."
- note added: "U35 TCA9538 at 0x70 controls D16 RGB; PC13 reset has a hardware pulldown."
- note removed: "17 / Status Indicators and Audible Alarm"
- note removed: "BUZZER_GATE"
- note removed: "BUZZER_LOW"
- note removed: "BZ1: active 3 V alarm. Q26 + R127 keep it off at reset; D18 clamps the switched lead."
- note removed: "U35: 3.3 V I2C GPIO at 0x70. Active-low RGB sinks; PC13 holds RESET low until board power is ready."
