File: dist/manufacturing/kicad-project/indicators.kicad_sch (KiCad schematic)
At the start: 9 parts, among them U35 TCA9538PWR

Commit message: Replace unavailable MCU and expander with stocked JLC parts
Use STM32G0B1CEU6 with a grounded UFQFPN48 exposed pad and a 512 KiB
firmware/readback target. Use PCA9538PWR with a PD-powered reset buffer,
bypass capacitor and pulldown to address independent-rail reset injection.

Regenerate local routing, native/manufacturing artifacts, assembly data,
stock evidence and the routed viewer. Preserve unrelated copper and holes
with the existing protected projection. Retain motion locks and physical
qualification holds. Preserve quoted DSN net names and native EP paste sizing.
Parts:
- removed U35: TCA9538PWR, TCA9538PWR, symbol Device:U_TCA9538PWR
- added C99: 100nF, capacitor_cap0603, symbol Device:capacitor_down
- added R137: 47kΩ, resistor_res0603, symbol Device:boxresistor_down
- added U35: PCA9538PWR, PCA9538PWR, symbol Device:U_PCA9538PWR
- added U37: SN74LVC1G17DBVR, SN74LVC1G17DBVR, symbol Device:U_SN74LVC1G17DBVR
Connections:
- net BUZZER_EN: now also U35.7 (P3)
- net GND: now also C99.2, R137.2, U35.1 (A0), U35.10 (P5), U35.11 (P6), U35.12 (P7), U35.2 (A1), U35.8 (GND), U35.9 (P4), U37.3 (GND)
- net PD_3V3: now also C99.1, U35.16 (VCC), U37.5 (VCC)
- net PD_SCL: now also U35.14 (SCL)
- net PD_SDA: now also U35.15 (SDA)
- net RGB_B_DRV: now also U35.6 (P2)
- net RGB_G_DRV: now also U35.5 (P1)
- net RGB_R_DRV: now also U35.4 (P0)
- net STATUS_GPIO: now also U37.2 (A)
- new net U35_RESET_N: R137.1, U35.3 (N_RESET), U37.4 (Y)
- no-connect marks 1 -> 2
Other:
- note added: "U35 PCA9538 at 0x70; U37 buffers PC13 reset into PD_3V3 with default-low bias."
- note added: "U35_RESET_N"
- note removed: "U35 TCA9538 at 0x70 controls D16 RGB; PC13 reset has a hardware pulldown."
