File: dist/manufacturing/kicad-project/pd_programming.kicad_sch (KiCad schematic)
At the start: 13 parts, among them U36 SN74LVC2G66DCUR

Commit message: Fix source warnings and organize schematic on A4 sheets
Parts:
- TP_EEP_SCL, TP_EEP_SDA, TP_PD_GND, TP_PD_ISO, TP_PD_VBUS, TP_PD_VREF, TP_PWR_GND, TP_VMOTOR: now not fitted; now left out of the parts list
Other:
- note added: "27 / PD Programming and Power Probes"
- note added: "U36 isolates both PD EEPROM I2Cc wires when TP_PD_ISO is grounded."
- note added: "Use fixed 5 V fixture power and a 3.3 V open-drain programmer; VREF is sense-only."
- note removed: "18 / PD Programming and Power Probes"
- note removed: "Program with fixed 5 V on J1, 3.3 V open-drain I2C and programmer VCC output OFF."
- note removed: "U36 isolates both I2Cc wires when TP_PD_ISO is grounded. Normal boot: pad released."
